File: electrical_hw/serial-port/serial.kicad_pcb (KiCad board)
At the start: 2 copper layers, 2 parts, among them U1 L78L05

Commit message: update
Parts:
- added 1: , Mounting_Holes:MountingHole_3.2mm_M3, F.Cu at (96.5, 19.1)
- added 3: , Mounting_Holes:MountingHole_3.2mm_M3, F.Cu at (54.6, 62.2)
- added 4: , Mounting_Holes:MountingHole_3.2mm_M3, F.Cu at (96.5, 62.2)
- added C1: .1, Capacitors_SMD:C_1206_HandSoldering, F.Cu at (63.5, 20.3)
- added C2: 10, Capacitors_THT:CP_Radial_D6.3mm_P2.50mm, F.Cu at (92.7, 29.2)
- added C3: .1, Capacitors_SMD:C_1206_HandSoldering, F.Cu at (83.8, 50.8)
- added C4: .1, Capacitors_SMD:C_1206_HandSoldering, F.Cu at (94.0, 53.3)
- added D1: RX, LEDs:LED_1206_HandSoldering, F.Cu at (72.4, 57.1)
- added D2: TX, LEDs:LED_1206_HandSoldering, F.Cu at (73.7, 39.4)
- added J1: 12V Pwr, Connectors:BARREL_JACK, F.Cu at (59.7, 31.8)
- added J2: Serial 5V, Pin_Headers:Pin_Header_Straight_1x04_Pitch2.54mm, F.Cu at (53.3, 43.2)
- added J3: XL-320, Connectors_Molex:Molex_MicroLatch-53253-0370_03x2.00mm_Straight, F.Cu at (97.8, 39.4)
- added J4: AX-12A, Connectors_Molex:Molex_SPOX-5267_22-03-5035_03x2.54mm_Straight, F.Cu at (97.8, 47.0)
- added R1: 330, Resistors_SMD:R_1206_HandSoldering, F.Cu at (85.1, 20.3)
- added R2: 1.8k, Resistors_SMD:R_1206_HandSoldering, F.Cu at (73.7, 20.3)
- added R3: 330, Resistors_SMD:R_1206_HandSoldering, F.Cu at (62.2, 57.1)
- added R4: 330, Resistors_SMD:R_1206_HandSoldering, F.Cu at (63.5, 39.4)
- added R5: 10k, Resistors_SMD:R_1206_HandSoldering, F.Cu at (76.2, 48.3)
- added U2: LM317, TO_SOT_Packages_THT:TO-220-3_Horizontal, F.Cu at (66.0, 27.9)
- added U3: 74LS126, Housings_SOIC:SOIC-14_3.9x8.7mm_Pitch1.27mm, F.Cu at (68.6, 48.3)
- 2: renamed from REF**; value MountingHole_3.2mm_M3 -> (none)
- U1: value L78L05 -> AP1117-50; footprint TO_SOT_Packages_THT:TO-92_Inline_Narrow_Oval -> TO_SOT_Packages_SMD:SOT-223-3_TabPin2
- moved 2 76.0 mm to (54.6, 19.1)
- moved U1 66.1 mm to (83.8, 43.2), turned to 90 degrees
Connections:
- U1 pad 1: +5V -> GND
- U1 pad 2: GND -> +5V
Routing:
- net GND: track 0.00 -> 149.1 mm
- net Net-(R5-Pad2): track 0.00 -> 109.7 mm, vias 0 -> 2
- net Net-(C1-Pad1): track 0.00 -> 67.4 mm
- net +8V: track 0.00 -> 65.4 mm, vias 0 -> 1
- net RXI: track 0.00 -> 50.6 mm, vias 0 -> 4
- net DATA: track 0.00 -> 46.5 mm, vias 0 -> 1
- net TXO: track 0.00 -> 35.9 mm, vias 0 -> 2
- net +5V: track 0.00 -> 29.9 mm, vias 0 -> 4
- net DTR: track 0.00 -> 22.8 mm, vias 0 -> 3
- net Net-(R1-Pad2): track 0.00 -> 21.3 mm
- net Net-(D2-Pad1): track 0.00 -> 6.16 mm
- net Net-(D1-Pad1): track 0.00 -> 6.16 mm
- net (no net): track 0.00 -> 0.54 mm
Other:
- net class High added: clearance 0.2, trace_width 0.75, via_dia 0.6, via_drill 0.4

Commit message: update
Parts:
- added D3: PWR, LEDs:LED_1206_HandSoldering, F.Cu at (80.0, 43.2)
- added R6: 330, Resistors_SMD:R_1206_HandSoldering, F.Cu at (80.0, 52.1)
- C1, C3, R1, R2, R5, U1, U3: moved to B.Cu
- moved 3 42.4 mm to (96.5, 55.9)
- moved 4 42.4 mm to (54.6, 55.9)
- moved C3 27.0 mm to (66.0, 30.5), turned to 270 degrees
- moved R1 21.6 mm to (63.5, 21.6)
- moved C1 16.6 mm to (80.0, 21.6), turned to 270 degrees
- moved U1 15.5 mm to (74.9, 30.5), turned to 0 degrees
- moved D2 15.3 mm to (62.2, 49.5), turned to 180 degrees
- moved R4 13.5 mm to (72.4, 49.5), turned to 0 degrees
- moved R2 10.9 mm to (63.5, 16.5)
- moved D1 10.5 mm to (62.2, 54.6), turned to 180 degrees
- moved R3 10.5 mm to (72.4, 54.6), turned to 0 degrees
- moved U2 10.2 mm to (71.1, 19.1)
- moved J3 10.2 mm to (87.6, 39.4), turned to 0 degrees
- moved U3 8.13 mm to (63.5, 41.9), turned to 0 degrees
- moved R5 7.18 mm to (71.1, 43.2), turned to 90 degrees
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Connections:
- C1 pad 1: Net-(C1-Pad1) -> +12V
- C2 pad 1: Net-(C1-Pad1) -> +12V
- J1 pad 1: Net-(C1-Pad1) -> +12V
- J3 pad 1: DATA -> GND
- J3 pad 3: GND -> DATA
- J4 pad 2: +8V -> +12V
- U1 pad 3: Net-(C1-Pad1) -> +12V
- U2 pad 3: Net-(C1-Pad1) -> +12V
Routing:
- net Net-(R5-Pad2): track 109.7 -> 15.4 mm, vias 2 -> 0
- net +12V: track 0.00 -> 73.0 mm
- net Net-(C1-Pad1): track 67.4 -> 0.00 mm
- net RXI: track 50.6 -> 20.3 mm, vias 4 -> 2
- net TXO: track 35.9 -> 22.2 mm, vias 2 -> 0
- net +5V: track 29.9 -> 39.1 mm, vias 4 -> 2
- net DTR: track 22.8 -> 16.1 mm, vias 3 -> 2
- net Net-(R1-Pad2): track 21.3 -> 14.9 mm
- net Net-(D3-Pad1): track 0.00 -> 4.89 mm
- net +8V: track 65.4 -> 62.1 mm
- net DATA: track 46.5 -> 43.8 mm, vias 1 -> 2
- net (no net): track 0.54 -> 1.27 mm
- net GND: track 149.1 -> 148.9 mm, vias 0 -> 1
- added copper zone on B.Cu, net GND
- added copper zone on F.Cu, net GND
Other:
- board outline added: 49.5 x 45.7 mm
- board text added: "Designed by Kevin Walchko 2018"
