File: electrical_hw/serial-port/serial.sch (KiCad schematic (older format))
At the start: 13 parts, among them J1 12V Pwr, J2 Serial 5V, J3 Servo, U1 L78L05, U2 LM317, U3 74LS126

Commit message: update
Parts:
- removed U1: L78L05, TO_SOT_Packages_THT:TO-92_Inline_Narrow_Oval, symbol L78L05_TO92
- added D1: RX, LEDs:LED_1206_HandSoldering, symbol LED
- added D2: TX, LEDs:LED_1206_HandSoldering, symbol LED
- added J3: XL-320, Connectors_Molex:Molex_MicroLatch-53253-0370_03x2.00mm_Straight, symbol Conn_01x03
- added R3, R4: 330, Resistors_SMD:R_1206_HandSoldering, symbol R
- added U1: AP1117-50, TO_SOT_Packages_SMD:SOT-223-3Lead_TabPin2, symbol AP1117-50
- J4: renamed from J3; value Servo -> AX-12A; footprint Pin_Headers:Pin_Header_Straight_1x03_Pitch2.54mm -> Connectors_Molex:Molex_SPOX-5267_22-03-5035_03x2.54mm_Straight
- renumbered R3 to R5
Connections:
- net +5V: now also U1.2 (VO)
- net +8V: now also J3.2 (Pin_2)
- net DATA: now also J3.1 (Pin_1)
- net GND: now also J3.3 (Pin_3), R3.2, R4.2, U1.1 (GND)
- net RXI: now also D1.2 (A)
- net TXO: now also D2.2 (A)
- net at C1.1, C2.1, J1.1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: now also U1.3 (VI)
- new net: D1.1 (K), R3.1
- new net: D2.1 (K), R4.1
Other:
- moved on the sheet: U3A, U3B
Changed lines of the file:
@@
 LIBS:contrib
 LIBS:valves
+LIBS:serial-cache
 EELAYER 25 0
 EELAYER END
@@
 L 74LS126 U3
 U 1 1 5A7F13E9
-P 5250 2250
-F 0 "U3" H 5350 2450 50  0000 C CNN
-F 1 "74LS126" H 5500 2100 50  0000 C CNN
-F 2 "Housings_SOIC:SOIC-14_3.9x8.7mm_Pitch1.27mm" H 5250 2250 50  0001 C CNN
-F 3 "" H 5250 2250 50  0001 C CNN
-	1    5250 2250
+P 5250 2150
+F 0 "U3" H 5350 2350 50  0000 C CNN
+F 1 "74LS126" H 5500 2000 50  0000 C CNN
+F 2 "Housings_SOIC:SOIC-14_3.9x8.7mm_Pitch1.27mm" H 5250 2150 50  0001 C CNN
+F 3 "" H 5250 2150 50  0001 C CNN
+	1    5250 2150
 	1    0    0    -1
 $EndComp
@@
 L 74LS126 U3
 U 2 1 5A7F1432
-P 5650 3100
-F 0 "U3" H 5750 3300 50  0000 C CNN
-F 1 "74LS126" H 5900 2950 50  0000 C CNN
-F 2 "Housings_SOIC:SOIC-14_3.9x8.7mm_Pitch1.27mm" H 5650 3100 50  0001 C CNN
-F 3 "" H 5650 3100 50  0001 C CNN
-	2    5650 3100
+P 5650 3700
+F 0 "U3" H 5750 3900 50  0000 C CNN
+F 1 "74LS126" H 5900 3550 50  0000 C CNN
+F 2 "Housings_SOIC:SOIC-14_3.9x8.7mm_Pitch1.27mm" H 5650 3700 50  0001 C CNN
+F 3 "" H 5650 3700 50  0001 C CNN
+	2    5650 3700
 	1    0    0    -1
 $EndComp
@@
 $EndComp
 $Comp
-L R R3
+L R R5
 U 1 1 5A7F169D
 P 8000 2850
-F 0 "R3" V 8080 2850 50  0000 C CNN
+F 0 "R5" V 8080 2850 50  0000 C CNN
 F 1 "10k" V 8000 2850 50  0000 C CNN
 F 2 "Resistors_SMD:R_1206_HandSoldering" V 7930 2850 50  0001 C CNN
@@
 $EndComp
 $Comp
-L L78L05_TO92 U1
-U 1 1 5A7F27F6
-P 3250 3000
-F 0 "U1" H 3100 3125 50  0000 C CNN
-F 1 "L78L05" H 3250 3125 50  0000 L CNN
-F 2 "TO_SOT_Packages_THT:TO-92_Inline_Narrow_Oval" H 3250 3225 50  0001 C CIN
-F 3 "" H 3250 2950 50  0001 C CNN
-	1    3250 3000
-	1    0    0    -1
-$EndComp
-$Comp
 L GND #PWR08
 U 1 1 5A7F28F9
@@
 Connection ~ 3250 3400
 $Comp
-L Conn_01x03 J3
+L Conn_01x03 J4
 U 1 1 5A7F2FF1
 P 7300 1300
-F 0 "J3" H 7300 1500 50  0000 C CNN
-F 1 "Servo" H 7300 1100 50  0000 C CNN
-F 2 "Pin_Headers:Pin_Header_Straight_1x03_Pitch2.54mm" H 7300 1300 50  0001 C CNN
+F 0 "J4" H 7300 1500 50  0000 C CNN
+F 1 "AX-12A" H 7300 1100 50  0000 C CNN
+F 2 "Connectors_Molex:Molex_SPOX-5267_22-03-5035_03x2.54mm_Straight" H 7300 1300 50  0001 C CNN
 F 3 "" H 7300 1300 50  0001 C CNN
 	1    7300 1300
 	1    0    0    -1
 $EndComp
-NoConn ~ 5200 3100
-NoConn ~ 5650 3400
-NoConn ~ 6100 3100
+NoConn ~ 5200 3700
+NoConn ~ 5650 4000
+NoConn ~ 6100 3700
 Text GLabel 5600 1200 2    60   Input ~ 0
 RXI
@@
 	1    0    0    -1
 $EndComp
-Text GLabel 6950 1200 0    60   BiDi ~ 0
+Text GLabel 6900 1200 0    60   BiDi ~ 0
 DATA
 $Comp
@@
 $EndComp
 Wire Wire Line
-	7100 1200 6950 1200
+	6900 1200 7100 1200
 Wire Wire Line
 	7100 1300 6500 1300
@@
 Wire Wire Line
 	6950 1400 6950 1450
-Text GLabel 5100 2650 0    60   Input ~ 0
+Text GLabel 5100 2550 0    60   Input ~ 0
 DTR
 Text GLabel 6550 2250 0    60   Input ~ 0
 TXO
-Text GLabel 5800 2250 2    60   Output ~ 0
+Text GLabel 5800 2150 2    60   Output ~ 0
 RXI
-Text GLabel 4700 2250 0    60   BiDi ~ 0
+Text GLabel 4700 2150 0    60   BiDi ~ 0
 DATA
 Text GLabel 7650 2250 2    60   BiDi ~ 0
@@
 	6550 2250 6650 2250
 Wire Wire Line
-	5700 2250 5800 2250
-Wire Wire Line
-	4700 2250 4800 2250
-Wire Wire Line
-	5100 2650 5250 2650
-Wire Wire Line
-	5250 2650 5250 2550
+	5700 2150 5800 2150
+Wire Wire Line
+	4700 2150 4800 2150
+Wire Wire Line
+	5100 2550 5250 2550
+Wire Wire Line
+	5250 2550 5250 2450
 Wire Wire Line
 	7100 2550 7100 2650
@@
 L GND #PWR014
 U 1 1 5A7F402D
-P 6500 3200
-F 0 "#PWR014" H 6500 2950 50  0001 C CNN
-F 1 "GND" H 6500 3050 50  0000 C CNN
-F 2 "" H 6500 3200 50  0001 C CNN
-F 3 "" H 6500 3200 50  0001 C CNN
-	1    6500 3200
-	1    0    0    -1
-$EndComp
-Wire Wire Line
-	6500 3200 6500 3100
+P 6500 3300
+F 0 "#PWR014" H 6500 3050 50  0001 C CNN
+F 1 "GND" H 6500 3150 50  0000 C CNN
+F 2 "" H 6500 3300 50  0001 C CNN
+F 3 "" H 6500 3300 50  0001 C CNN
+	1    6500 3300
+	1    0    0    -1
+$EndComp
+Wire Wire Line
+	6500 3100 6500 3300
 Wire Wire Line
 	6500 3100 6600 3100
@@
 	1    0    0    -1
 $EndComp
+$Comp
+L LED D1
+U 1 1 5A862706
+P 5750 2450
+F 0 "D1" H 5750 2550 50  0000 C CNN
+F 1 "RX" H 5750 2350 50  0000 C CNN
+F 2 "LEDs:LED_1206_HandSoldering" H 5750 2450 50  0001 C CNN
+F 3 "" H 5750 2450 50  0001 C CNN
+	1    5750 2450
+	0    -1   -1   0
+$EndComp
+$Comp
+L LED D2
+U 1 1 5A862765
+P 6300 2600
+F 0 "D2" H 6300 2700 50  0000 C CNN
+F 1 "TX" H 6300 2500 50  0000 C CNN
+F 2 "LEDs:LED_1206_HandSoldering" H 6300 2600 50  0001 C CNN
+F 3 "" H 6300 2600 50  0001 C CNN
+	1    6300 2600
+	0    -1   -1   0
+$EndComp
+$Comp
+L R R3
+U 1 1 5A8627B6
+P 5750 2850
+F 0 "R3" V 5830 2850 50  0000 C CNN
+F 1 "330" V 5750 2850 50  0000 C CNN
+F 2 "Resistors_SMD:R_1206_HandSoldering" V 5680 2850 50  0001 C CNN
+F 3 "" H 5750 2850 50  0001 C CNN
+	1    5750 2850
+	1    0    0    -1
+$EndComp
+$Comp
+L GND #PWR016
+U 1 1 5A8628F6
+P 5750 3100
+F 0 "#PWR016" H 5750 2850 50  0001 C CNN
+F 1 "GND" H 5750 2950 50  0000 C CNN
+F 2 "" H 5750 3100 50  0001 C CNN
+F 3 "" H 5750 3100 50  0001 C CNN
+	1    5750 3100
+	1    0    0    -1
+$EndComp
+Wire Wire Line
+	5750 2300 5750 2150
+Connection ~ 5750 2150
+Wire Wire Line
+	5750 2600 5750 2700
+Wire Wire Line
+	5750 3000 5750 3100
+$Comp
+L R R4
+U 1 1 5A862D7C
+P 6300 3000
+F 0 "R4" V 6380 3000 50  0000 C CNN
+F 1 "330" V 6300 3000 50  0000 C CNN
+F 2 "Resistors_SMD:R_1206_HandSoldering" V 6230 3000 50  0001 C CNN
+F 3 "" H 6300 3000 50  0001 C CNN
+	1    6300 3000
+	1    0    0    -1
+$EndComp
+Wire Wire Line
+	6300 2450 6300 2400
+Wire Wire Line
+	6300 2400 6600 2400
+Wire Wire Line
+	6600 2400 6600 2250
+Connection ~ 6600 2250
+Wire Wire Line
+	6300 2750 6300 2850
+Wire Wire Line
+	6300 3150 6300 3200
+Wire Wire Line
+	6300 3200 6500 3200
+Connection ~ 6500 3200
+$Comp
+L Conn_01x03 J3
+U 1 1 5A863A11
+P 7300 750
+F 0 "J3" H 7300 950 50  0000 C CNN
+F 1 "XL-320" H 7300 550 50  0000 C CNN
+F 2 "Connectors_Molex:Molex_MicroLatch-53253-0370_03x2.00mm_Straight" H 7300 750 50  0001 C CNN
+F 3 "" H 7300 750 50  0001 C CNN
+	1    7300 750
+	1    0    0    -1
+$EndComp
+Wire Wire Line
+	7100 850  7050 850
+Wire Wire Line
+	7050 850  7050 1400
+Connection ~ 7050 1400
+Wire Wire Line
+	7100 750  7000 750
+Wire Wire Line
+	7000 750  7000 1300
+Connection ~ 7000 1300
+Wire Wire Line
+	7100 650  6950 650
+Wire Wire Line
+	6950 650  6950 1200
+Connection ~ 6950 1200
+$Comp
+L AP1117-50 U1
+U 1 1 5A864FB2
+P 3250 3000
+F 0 "U1" H 3100 3125 50  0000 C CNN
+F 1 "AP1117-50" H 3250 3125 50  0000 L CNN
+F 2 "TO_SOT_Packages_SMD:SOT-223-3Lead_TabPin2" H 3250 3200 50  0001 C CNN
+F 3 "" H 3350 2750 50  0001 C CNN
+	1    3250 3000
+	1    0    0    -1
+$EndComp
+$Comp
+L PWR_FLAG #FLG017
+U 1 1 5A864DA9
+P 5150 3200
+F 0 "#FLG017" H 5150 3275 50  0001 C CNN
+F 1 "PWR_FLAG" H 5150 3350 50  0000 C CNN
+F 2 "" H 5150 3200 50  0001 C CNN
+F 3 "" H 5150 3200 50  0001 C CNN
+	1    5150 3200
+	-1   0    0    1
+$EndComp
+$Comp
+L +5V #PWR018
+U 1 1 5A864DF3
+P 5150 3050
+F 0 "#PWR018" H 5150 2900 50  0001 C CNN
+F 1 "+5V" H 5150 3190 50  0000 C CNN
+F 2 "" H 5150 3050 50  0001 C CNN
+F 3 "" H 5150 3050 50  0001 C CNN
+	1    5150 3050
+	1    0    0    -1
+$EndComp
+Wire Wire Line
+	5150 3050 5150 3200
 $EndSCHEMATC

Commit message: update
Parts:
- added D3: PWR, LEDs:LED_1206_HandSoldering, symbol LED
- added R6: 330, Resistors_SMD:R_1206_HandSoldering, symbol R
Connections:
- net +5V: now also D3.2 (A)
- net +8V: no longer J4.2 (Pin_2)
- net DATA: now also J3.3 (Pin_3); no longer J3.1 (Pin_1)
- net GND: now also J3.1 (Pin_1), R6.2; no longer J3.3 (Pin_3)
- net +12V: now reaches C1.1, C2.1, J1.1, U1.3 (VI), U2.3 (VI)
- net +12V: now also J4.2 (Pin_2)
- new net: D3.1 (K), R6.1
Other:
- moved on the sheet: J1, J2, J3, J4, U3B
