File: ax12/electrical/power/robot.kicad_pcb (KiCad board)
At the start: 2 copper layers, 99.1 x 47 mm, 38 parts, among them J1 12V, J2 LEG1, J3 Pi USB Pwr, J4 Serial, J5 LEG2, J6 LEG3, J7 LEG4, J8 Data P, J9 Data S, U1 LM317_12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

Commit message: update
Parts:
- removed D2: RX, LEDs:LED_D5.0mm
- removed D3: PWR, LEDs:LED_1206_HandSoldering
- removed J7: LEG4, Connectors_Molex:Molex_MicroLatch-53253-0370_03x2.00mm_Straight
- removed J8: Data P, Pin_Headers:Pin_Header_Straight_1x03_Pitch2.54mm
- removed J9: Data S, Pin_Headers:Pin_Header_Straight_1x03_Pitch2.54mm
- removed REF1, REF2, REF3, REF5, REF6, REF7, REF8: , Mounting_Holes:MountingHole_3.2mm_M3
- removed REF4: 3.2mm_M3, Mounting_Holes:MountingHole_3.2mm_M3
- added ?: , Mounting_Holes:MountingHole_2.7mm, F.Cu at (154.9, 63.5)
- added ?: , Mounting_Holes:MountingHole_2.7mm, F.Cu at (113.0, 63.5)
- added ?: , Mounting_Holes:MountingHole_2.7mm, F.Cu at (113.0, 105.4)
- added ?: , Mounting_Holes:MountingHole_2.7mm, F.Cu at (154.9, 105.4)
- added ?: , Symbols:OSHW-Logo_7.5x8mm_SilkScreen, B.Cu at (121.9, 66.0)
- added C7: C, Capacitors_SMD:C_1206_HandSoldering, B.Cu at (130.8, 101.6)
- added C8: C, Capacitors_SMD:C_1206_HandSoldering, B.Cu at (143.5, 101.6)
- added R9: 330, Resistors_SMD:R_1206_HandSoldering, F.Cu at (123.2, 95.2)
- C5, C6: value C -> .1; footprint Capacitors_SMD:C_1206_HandSoldering -> Capacitors_THT:CP_Radial_D6.3mm_P2.50mm; moved to F.Cu
- D1: value TX -> PWR; footprint LEDs:LED_D5.0mm -> LEDs:LED_1206_HandSoldering
- J1: value 12V -> LEG1; footprint TerminalBlocks_Phoenix:TerminalBlock_Phoenix_PT-3.5mm_2pol -> Connectors_Molex:Molex_SPOX-5267_22-03-5035_03x2.54mm_Straight
- J2: value LEG1 -> LEG2; footprint Connectors_Molex:Molex_MicroLatch-53253-0370_03x2.00mm_Straight -> Connectors_Molex:Molex_SPOX-5267_22-03-5035_03x2.54mm_Straight
- J3: value Pi USB Pwr -> LEG4; footprint Pin_Headers:Pin_Header_Straight_1x02_Pitch2.54mm -> Connectors_Molex:Molex_SPOX-5267_22-03-5035_03x2.54mm_Straight
- J4: value Serial -> LEG3; footprint Pin_Headers:Pin_Header_Straight_1x04_Pitch2.54mm -> Connectors_Molex:Molex_SPOX-5267_22-03-5035_03x2.54mm_Straight
- J5: value LEG2 -> Data P; footprint Connectors_Molex:Molex_MicroLatch-53253-0370_03x2.00mm_Straight -> Pin_Headers:Pin_Header_Straight_1x03_Pitch2.54mm
- J6: value LEG3 -> PWR IN; footprint Connectors_Molex:Molex_MicroLatch-53253-0370_03x2.00mm_Straight -> TerminalBlocks_Phoenix:TerminalBlock_Phoenix_PT-3.5mm_2pol
- R1, R3: value 330 -> 390
- R2, R4: value 1.8k -> 3.3k
- R5: value 10k -> 390; moved to B.Cu
- R6, R8: value 330 -> 3.3k; moved to B.Cu
- R7: value 330 -> 390; moved to B.Cu
- U2: value AP1117-50 -> LM317_12; footprint TO_SOT_Packages_SMD:SOT-223-3_TabPin2 -> TO_SOT_Packages_THT:TO-220-3_Horizontal; moved to F.Cu
- U3: value 74LS126 -> LM317_34; footprint Housings_SOIC:SOIC-14_3.9x8.7mm_Pitch1.27mm -> TO_SOT_Packages_THT:TO-220-3_Horizontal
- moved J4 94.3 mm to (156.2, 86.4)
- moved U3 57.8 mm to (133.3, 88.9)
- moved R5 55.3 mm to (130.8, 97.8)
- moved R7 53.1 mm to (143.5, 97.8), turned to 0 degrees
- moved C4 44.9 mm to (154.9, 72.4), turned to 180 degrees
- moved C3 43.3 mm to (114.3, 71.1), turned to 180 degrees
- moved R6 41.8 mm to (130.8, 92.7), turned to 180 degrees
- moved D1 39.2 mm to (119.4, 95.2), turned to 90 degrees
- moved C6 37.0 mm to (154.9, 94.0), turned to 180 degrees
- moved J3 34.5 mm to (116.8, 86.4)
- moved J1 31.9 mm to (116.8, 80.0), turned to 180 degrees
- moved C5 28.5 mm to (114.3, 95.2), turned to 180 degrees
- moved R3 26.9 mm to (142.2, 67.3)
- moved J2 25.7 mm to (156.2, 80.0), turned to 180 degrees
- moved U4 24.2 mm to (144.8, 88.9), turned to 180 degrees
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Connections:
- C1 pad 1: +12V -> +VDC
- C2 pad 1: +5V -> +VDC
- C3 pad 1: /PWR12 -> Net-(C3-Pad1)
- C4 pad 1: /PWR34 -> Net-(C4-Pad1)
- C5 pad 1: +12V -> Net-(C5-Pad1)
- C6 pad 1: +12V -> Net-(C6-Pad1)
- D1 pad 1: GND -> GNDA
- J1 pad 1: GNDA -> DATA
- J1 pad 2: +12V -> Net-(C3-Pad1)
- J2 pad 1: GNDA -> DATA
- J2 pad 2: /PWR12 -> Net-(C4-Pad1)
- J2 pad 3: /DATA -> GNDA
- J3 pad 1: GNDA -> DATA
- J3 pad 2: +5V -> Net-(C5-Pad1)
- J4 pad 1: GND -> DATA
- J4 pad 2: /DTR -> Net-(C6-Pad1)
- J4 pad 3: /RXO -> GNDA
- J5 pad 2: /PWR12 -> DATA
- J5 pad 3: /DATA -> +VDC
- J6 pad 2: /PWR34 -> +VDC
- R1 pad 1: /PWR12 -> Net-(C3-Pad1)
- R3 pad 1: /PWR34 -> Net-(C4-Pad1)
- R5 pad 1: +5VA -> Net-(C5-Pad1)
- R6 pad 1: Net-(D1-Pad2) -> Net-(R5-Pad2)
- R6 pad 2: /TXI -> GNDA
- R7 pad 1: Net-(D2-Pad2) -> Net-(C6-Pad1)
- R7 pad 2: /RXO -> Net-(R7-Pad2)
- R8 pad 1: +5V -> Net-(R7-Pad2)
- R8 pad 2: Net-(D3-Pad2) -> GNDA
- U1 pad 2: +12V -> +VDC
- U1 pad 3: /PWR12 -> Net-(C3-Pad1)
- U2 pad 1: GNDA -> Net-(R3-Pad2)
- U2 pad 2: +5V -> +VDC
- U2 pad 3: +12V -> Net-(C4-Pad1)
- U3 pad 1: /DTR -> Net-(R5-Pad2)
- U3 pad 2: Net-(J9-Pad2) -> +VDC
- U3 pad 3: /RXO -> Net-(C5-Pad1)
- U4 pad 1: Net-(R3-Pad2) -> Net-(R7-Pad2)
- U4 pad 2: +12V -> +VDC
- U4 pad 3: /PWR34 -> Net-(C6-Pad1)
Routing:
- net +12V: track 71.5 -> 0.00 mm, vias 2 -> 0
- net DATA: track 0.00 -> 60.7 mm
- net /RXO: track 51.3 -> 0.00 mm, vias 1 -> 0
- net +5V: track 49.5 -> 0.00 mm, vias 2 -> 0
- net GND: track 49.4 -> 0.00 mm, vias 3 -> 0
- net /DATA: track 48.8 -> 0.00 mm, vias 1 -> 0
- net +VDC: track 0.00 -> 48.6 mm
- net Net-(C3-Pad1): track 0.00 -> 47.6 mm
- net /TXI: track 40.1 -> 0.00 mm
- net /PWR12: track 35.6 -> 0.00 mm
- net /PWR34: track 34.3 -> 0.00 mm
- net Net-(R5-Pad2): track 30.0 -> 0.00 mm
- net Net-(J9-Pad2): track 29.4 -> 0.00 mm, vias 1 -> 0
- net Net-(C6-Pad1): track 0.00 -> 27.5 mm
- net Net-(C5-Pad1): track 0.00 -> 26.5 mm
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Other:
- board size 99.1 x 47 mm -> 49.5 x 49.5 mm
- net class large: trace_width 0.6 -> 1.6
- board text added: "V D G"
- board text added: "Walchko (c) 2018"

Commit message: up
Parts:
- ?: moved to F.Cu
- C3, C4, C5, C6: footprint Capacitors_THT:CP_Radial_D6.3mm_P2.50mm -> Capacitors_SMD:C_1206_HandSoldering; moved to B.Cu
- moved J6 41.0 mm to (154.9, 86.4), turned to 90 degrees
- moved D1 34.1 mm to (133.3, 64.1), turned to 270 degrees
- moved J5 26.9 mm to (111.8, 87.0), turned to 180 degrees
- moved R9 24.4 mm to (133.3, 73.0), turned to 270 degrees
- moved ? 18.5 mm to (133.3, 80.6), turned to 0 degrees
- moved J3 11.4 mm to (113.0, 97.2), turned to 90 degrees
- moved R5 10.6 mm to (120.7, 101.0)
- moved R2 9.94 mm to (120.7, 67.9)
- moved C8 9.03 mm to (137.8, 94.6), turned to 180 degrees
- moved R8 9.03 mm to (137.8, 99.7)
- moved R6 8.47 mm to (128.9, 101.0), turned to 0 degrees
- moved J2 8.35 mm to (154.9, 71.8), turned to 270 degrees
- moved C4 8.35 mm to (146.7, 73.7)
- moved C6 8.28 mm to (146.7, 94.6)
- moved C7 7.24 mm to (128.9, 94.6), turned to 0 degrees
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Routing:
- net +VDC: track 48.6 -> 110.4 mm, vias 0 -> 3
- net DATA: track 60.7 -> 95.1 mm, vias 0 -> 1
- net GNDA: track 136.7 -> 164.8 mm, vias 3 -> 5
- net Net-(C3-Pad1): track 47.6 -> 65.2 mm, vias 0 -> 4
- net Net-(R1-Pad2): track 0.00 -> 16.0 mm, vias 0 -> 1
- net Net-(R5-Pad2): track 0.00 -> 15.8 mm, vias 0 -> 1
- net Net-(R7-Pad2): track 0.00 -> 15.1 mm, vias 0 -> 1
- net Net-(R3-Pad2): track 8.22 -> 16.7 mm, vias 0 -> 1
- net Net-(C5-Pad1): track 26.5 -> 18.7 mm
- net Net-(D1-Pad2): track 3.81 -> 9.94 mm
- net Net-(C4-Pad1): track 23.2 -> 20.3 mm, vias 1 -> 0
- net Net-(C6-Pad1): track 27.5 -> 27.8 mm, vias 0 -> 1

Commit message: updates
Routing:
- net GNDA: track 164.8 -> 0.00 mm, vias 5 -> 0
- net Net-(C3-Pad1): track 65.2 -> 45.6 mm, vias 4 -> 1
- net DATA: track 95.1 -> 107.1 mm, vias 1 -> 0
- net Net-(C6-Pad1): track 27.8 -> 36.5 mm, vias 1 -> 0
- net Net-(R5-Pad2): track 15.8 -> 24.3 mm, vias 1 -> 0
- net Net-(C4-Pad1): track 20.3 -> 27.7 mm
- net Net-(C5-Pad1): track 18.7 -> 26.0 mm
- net +VDC: track 110.4 -> 107.2 mm, vias 3 -> 1
- added copper zone on B.Cu, net GNDA
- added copper zone on F.Cu, net GNDA
