File: ax12/electrical/power/robot.sch (KiCad schematic (older format))
At the start: 30 parts, among them J1 12V, J2 LEG1, J3 Pi USB Pwr, J4 Serial, J5 LEG2, J6 LEG3, J7 LEG4, J8 Data P, J9 Data S, U1 LM317_12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

Commit message: update
Parts:
- removed C1: C, Capacitors_SMD:C_1206_HandSoldering, symbol C
- removed D1: TX, LEDs:LED_D5.0mm, symbol LED
- removed D2: RX, LEDs:LED_D5.0mm, symbol LED
- removed J3: Pi USB Pwr, Pin_Headers:Pin_Header_Straight_1x02_Pitch2.54mm, symbol Conn_01x02
- removed J4: Serial, Pin_Headers:Pin_Header_Straight_1x04_Pitch2.54mm, symbol Conn_01x04
- removed J5: LEG2, Connectors_Molex:Molex_MicroLatch-53253-0370_03x2.00mm_Straight, symbol Conn_01x03
- removed J7: LEG4, Connectors_Molex:Molex_MicroLatch-53253-0370_03x2.00mm_Straight, symbol Conn_01x03
- removed J9: Data S, Pin_Headers:Pin_Header_Straight_1x03_Pitch2.54mm, symbol Conn_01x03
- removed R7: 330, Resistors_SMD:R_1206_HandSoldering, symbol R
- removed U2: AP1117-50, TO_SOT_Packages_SMD:SOT-223-3_TabPin2, symbol AP1117-50
- removed U3: 74LS126, Housings_SOIC:SOIC-14_3.9x8.7mm_Pitch1.27mm, symbol 74LS126
- added C4, C5: .1, Capacitors_THT:CP_Radial_D6.3mm_P2.50mm, symbol CP
- added C7: C, Capacitors_SMD:C_1206_HandSoldering, symbol C
- added J2: LEG2, Connectors_Molex:Molex_SPOX-5267_22-03-5035_03x2.54mm_Straight, symbol Conn_01x03
- added J3: LEG4, Connectors_Molex:Molex_SPOX-5267_22-03-5035_03x2.54mm_Straight, symbol Conn_01x03
- added R3: 390, Resistors_SMD:R_1206_HandSoldering, symbol R
- added R4: 3.3k, Resistors_SMD:R_1206_HandSoldering, symbol R
- added U2: LM317_12, TO_SOT_Packages_THT:TO-220-3_Horizontal, symbol LM317_TO3
- added U3: LM317_34, TO_SOT_Packages_THT:TO-220-3_Horizontal, symbol LM317_TO3
- J1: renamed from J2; footprint Connectors_Molex:Molex_MicroLatch-53253-0370_03x2.00mm_Straight -> Connectors_Molex:Molex_SPOX-5267_22-03-5035_03x2.54mm_Straight
- J4: renamed from J6; footprint Connectors_Molex:Molex_MicroLatch-53253-0370_03x2.00mm_Straight -> Connectors_Molex:Molex_SPOX-5267_22-03-5035_03x2.54mm_Straight
- J6: renamed from J1; value 12V -> PWR IN
- R1: value 330 -> 390
- R2: value 1.8k -> 3.3k
- R5: value 10k -> 390
- R6: value 330 -> 3.3k
- R7: renamed from R3; value 330 -> 390
- R8: renamed from R4; value 1.8k -> 3.3k
- renumbered C5 to C1, C4 to C6, C6 to C8, D3 to D1, J8 to J5, R8 to R9
Connections:
- net +5V is gone; now on net +VDC: C2.1, J5.3 (Pin_3), R9.1
- net TXI is gone; now on net GNDA: R6.2
- net DATA: now also J1.1 (Pin_1), J4.1 (Pin_1), J2.1 (Pin_1), J3.1 (Pin_1); no longer J1.3 (Pin_3), J4.3 (Pin_3)
- net GNDA: now also J1.3 (Pin_3), J4.3 (Pin_3), C4.2, C5.2, C7.2, J2.3 (Pin_3), J3.3 (Pin_3), R4.2; no longer J1.1 (Pin_1), J4.1 (Pin_1)
- net at R5.2: now also R6.1, U3.1 (ADJ)
- net +12V renamed +VDC
- net +VDC: now also C7.1, U2.2 (VI), U3.2 (VI)
- net +5VA: no longer names the net of R5.1
- net +5VA: now also C5.1, J3.2 (Pin_2), U3.3 (VO)
- net PWR12: no longer names the net of C3.1, J1.2 (Pin_2), R1.1, U1.3 (VO)
- net PWR34: no longer names the net of C6.1, J4.2 (Pin_2), R7.1, U4.3 (VO)
- new net: R3.2, R4.1, U2.1 (ADJ)
- new net: C4.1, J2.2 (Pin_2), R3.1, U2.3 (VO)
- no-connect marks 3 -> 0
Other:
- note removed: "DATA"
- note removed: "XL-320 Servo Data to Serial Converter"
- moved on the sheet: C1, C3, C6, C8, D1, J1, J4, J5, J6, R1, R2, R7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

Commit message: up
Parts:
- C3, C4, C5, C6: footprint Capacitors_THT:CP_Radial_D6.3mm_P2.50mm -> Capacitors_SMD:C_1206_HandSoldering
Changed lines of the file:
@@
 F 0 "C3" H 4525 3850 50  0000 L CNN
 F 1 ".1" H 4525 3650 50  0000 L CNN
-F 2 "Capacitors_THT:CP_Radial_D6.3mm_P2.50mm" H 4538 3600 50  0001 C CNN
+F 2 "Capacitors_SMD:C_1206_HandSoldering" H 4538 3600 50  0001 C CNN
 F 3 "" H 4500 3750 50  0001 C CNN
 	1    4500 3750
@@
 F 0 "C6" H 6925 3750 50  0000 L CNN
 F 1 ".1" H 6925 3550 50  0000 L CNN
-F 2 "Capacitors_THT:CP_Radial_D6.3mm_P2.50mm" H 6938 3500 50  0001 C CNN
+F 2 "Capacitors_SMD:C_1206_HandSoldering" H 6938 3500 50  0001 C CNN
 F 3 "" H 6900 3650 50  0001 C CNN
 	1    6900 3650
@@
 F 0 "C4" H 4525 5700 50  0000 L CNN
 F 1 ".1" H 4525 5500 50  0000 L CNN
-F 2 "Capacitors_THT:CP_Radial_D6.3mm_P2.50mm" H 4538 5450 50  0001 C CNN
+F 2 "Capacitors_SMD:C_1206_HandSoldering" H 4538 5450 50  0001 C CNN
 F 3 "" H 4500 5600 50  0001 C CNN
 	1    4500 5600
@@
 F 0 "C5" H 6475 5650 50  0000 L CNN
 F 1 ".1" H 6475 5450 50  0000 L CNN
-F 2 "Capacitors_THT:CP_Radial_D6.3mm_P2.50mm" H 6488 5400 50  0001 C CNN
+F 2 "Capacitors_SMD:C_1206_HandSoldering" H 6488 5400 50  0001 C CNN
 F 3 "" H 6450 5550 50  0001 C CNN
 	1    6450 5550

Commit message: updates
Changed lines of the file:
@@
 Wire Notes Line
 	2950 4900 2950 2250
-Text Notes 3000 2200 0    60   ~ 0
+Text Notes 3400 700  0    60   ~ 0
 Power System and Servo Bus Interface
 $Comp
