File: ax12/electrical/power-v2/robot.sch (KiCad schematic (older format))
At the start: 28 parts, among them J1 LEG1, J2 LEG2, J3 LEG4, J4 LEG3, J5 Data P, J6 PWR IN, U1 LM317_12, U2 LM317_12, U3 LM317_34, U4 LM317_34

Commit message: new power board
Parts:
- removed C7, C8: C, Capacitors_SMD:C_1206_HandSoldering, symbol C
- removed R1, R3, R5, R7: 390, Resistors_SMD:R_1206_HandSoldering, symbol R
- removed R2, R4, R6, R8: 3.3k, Resistors_SMD:R_1206_HandSoldering, symbol R
- removed U1, U2: LM317_12, TO_SOT_Packages_THT:TO-220-3_Horizontal, symbol LM317_TO3
- removed U3, U4: LM317_34, TO_SOT_Packages_THT:TO-220-3_Horizontal, symbol LM317_TO3
- added J7: EXT, Connectors_Molex:Molex_SPOX-5267_22-03-5035_03x2.54mm_Straight, symbol Conn_01x03
- added J8: USB, TerminalBlocks_Phoenix:TerminalBlock_Phoenix_PT-3.5mm_2pol, symbol Screw_Terminal_01x02
- added U1: AP1117-50, ksmd:SOT-223-3_TabPin2, symbol AP1117-50
- C3, C4, C5, C6: footprint Capacitors_SMD:C_1206_HandSoldering -> Capacitors_THT:CP_Radial_D6.3mm_P2.50mm
- J3: value LEG4 -> LEG3
- J4: value LEG3 -> LEG4
- J5: footprint Pin_Headers:Pin_Header_Straight_1x03_Pitch2.54mm -> Pin_Headers:Pin_Header_Straight_1x02_Pitch2.54mm; symbol Conn_01x03 -> Conn_01x02
- R9: value 330 -> 3.3k
Connections:
- net DATA: now also J7.1 (Pin_1)
- net +12V: now reaches C3.1, J1.2 (Pin_2)
- net +12V: now also C2.1, C4.1, C5.1, C6.1, J2.2 (Pin_2), J3.2 (Pin_2), J4.2 (Pin_2), J6.2 (Pin_2), R9.1, J7.2 (Pin_2), U1.3 (VI)
- removed net +VDC: C1.1, C2.1, J5.3 (Pin_3), J6.2 (Pin_2), R9.1
- net GNDA renamed GND
- net GND: now also J7.3 (Pin_3), J8.1 (Pin_1), U1.1 (GND)
- new net +5V: C1.1, J8.2 (Pin_2), U1.2 (VO)
Other:
- moved on the sheet: C1, C3, C4, C5, C6, D1, J1, J2, J3, J4, J6, R9
