File: ax12/electrical/power-v3/robot.sch (KiCad schematic (older format))
At the start: 22 parts, among them J1 LEG1, J10 PWR, J11 GND, J12 GND, J13 GND, J2 LEG2, J3 LEG3, J4 LEG4, J5 Data P, J6 PWR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

Commit message: power 3 done :tada: :electric_plug:
Other:
- note added: "AX-12A Servo Interface"
- note added: "External 12V Power System"
- note added: "Power Flags"
- note added: "USB 5V Power System"
- note removed: "Power System and Servo Bus Interface"
- moved on the sheet: C1, C2, C3, C4, C5, C6, D1, J1, J10, J11, J12, J13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

Commit message: update
Changed lines of the file:
@@
 L PWR_FLAG #FLG01
 U 1 1 5A7F9C06
-P 2450 6900
-F 0 "#FLG01" H 2450 6975 50  0001 C CNN
-F 1 "PWR_FLAG" H 2450 7050 50  0000 C CNN
-F 2 "" H 2450 6900 50  0001 C CNN
-F 3 "" H 2450 6900 50  0001 C CNN
-	1    2450 6900
+P 1900 6550
+F 0 "#FLG01" H 1900 6625 50  0001 C CNN
+F 1 "PWR_FLAG" H 1900 6700 50  0000 C CNN
+F 2 "" H 1900 6550 50  0001 C CNN
+F 3 "" H 1900 6550 50  0001 C CNN
+	1    1900 6550
 	1    0    0    -1
 $EndComp
@@
 L PWR_FLAG #FLG02
 U 1 1 5A935890
-P 1550 6900
-F 0 "#FLG02" H 1550 6975 50  0001 C CNN
-F 1 "PWR_FLAG" H 1550 7050 50  0000 C CNN
-F 2 "" H 1550 6900 50  0001 C CNN
-F 3 "" H 1550 6900 50  0001 C CNN
-	1    1550 6900
+P 1250 6650
+F 0 "#FLG02" H 1250 6725 50  0001 C CNN
+F 1 "PWR_FLAG" H 1250 6800 50  0000 C CNN
+F 2 "" H 1250 6650 50  0001 C CNN
+F 3 "" H 1250 6650 50  0001 C CNN
+	1    1250 6650
 	-1   0    0    1
 $EndComp
@@
 L +12V #PWR05
 U 1 1 5AA56F03
-P 1550 6800
-F 0 "#PWR05" H 1550 6650 50  0001 C CNN
-F 1 "+12V" H 1550 6940 50  0000 C CNN
-F 2 "" H 1550 6800 50  0001 C CNN
-F 3 "" H 1550 6800 50  0001 C CNN
-	1    1550 6800
+P 1250 6550
+F 0 "#PWR05" H 1250 6400 50  0001 C CNN
+F 1 "+12V" H 1250 6690 50  0000 C CNN
+F 2 "" H 1250 6550 50  0001 C CNN
+F 3 "" H 1250 6550 50  0001 C CNN
+	1    1250 6550
 	1    0    0    -1
 $EndComp
@@
 L GND #PWR012
 U 1 1 5AA58E71
-P 2450 7000
-F 0 "#PWR012" H 2450 6750 50  0001 C CNN
-F 1 "GND" H 2450 6850 50  0000 C CNN
-F 2 "" H 2450 7000 50  0001 C CNN
-F 3 "" H 2450 7000 50  0001 C CNN
-	1    2450 7000
+P 1900 6650
+F 0 "#PWR012" H 1900 6400 50  0001 C CNN
+F 1 "GND" H 1900 6500 50  0000 C CNN
+F 2 "" H 1900 6650 50  0001 C CNN
+F 3 "" H 1900 6650 50  0001 C CNN
+	1    1900 6650
 	1    0    0    -1
 $EndComp
@@
 L PWR_FLAG #FLG013
 U 1 1 5AA58FA3
-P 3150 7050
-F 0 "#FLG013" H 3150 7125 50  0001 C CNN
-F 1 "PWR_FLAG" H 3150 7200 50  0000 C CNN
-F 2 "" H 3150 7050 50  0001 C CNN
-F 3 "" H 3150 7050 50  0001 C CNN
-	1    3150 7050
+P 2600 6650
+F 0 "#FLG013" H 2600 6725 50  0001 C CNN
+F 1 "PWR_FLAG" H 2600 6800 50  0000 C CNN
+F 2 "" H 2600 6650 50  0001 C CNN
+F 3 "" H 2600 6650 50  0001 C CNN
+	1    2600 6650
 	-1   0    0    1
 $EndComp
@@
 L +5V #PWR014
 U 1 1 5AA58FDB
-P 3150 6950
-F 0 "#PWR014" H 3150 6800 50  0001 C CNN
-F 1 "+5V" H 3150 7090 50  0000 C CNN
-F 2 "" H 3150 6950 50  0001 C CNN
-F 3 "" H 3150 6950 50  0001 C CNN
-	1    3150 6950
+P 2600 6550
+F 0 "#PWR014" H 2600 6400 50  0001 C CNN
+F 1 "+5V" H 2600 6690 50  0000 C CNN
+F 2 "" H 2600 6550 50  0001 C CNN
+F 3 "" H 2600 6550 50  0001 C CNN
+	1    2600 6550
 	1    0    0    -1
 $EndComp
@@
 	5500 3750 5500 3850
 Wire Wire Line
-	1550 6900 1550 6800
+	1250 6650 1250 6550
 Wire Wire Line
 	5500 4150 5500 4200
@@
 	4900 2050 4900 2000
 Wire Wire Line
-	2450 7000 2450 6900
-Wire Wire Line
-	3150 7050 3150 6950
+	1900 6650 1900 6550
+Wire Wire Line
+	2600 6650 2600 6550
 Wire Wire Line
 	6700 1550 7550 1550
