File: ax12/electrical/power-v3/robot.kicad_pcb (KiCad board)
At the start: 2 copper layers, 38.7 x 39.4 mm, 27 parts, among them J1 LEG1, J10 PWR, J11 GND, J12 GND, J13 GND, J2 LEG2, J3 LEG3, J4 LEG4, J5 Data P, J6 PWR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

Commit message: update
Other:
- board text added: "Ver 3"
Changed lines of the file:
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@@
     (area 102.202857 54.27 155.607143 103.945)
     (thickness 1.6)
-    (drawings 8)
+    (drawings 9)
     (tracks 73)
     (zones 0)
@@
       (effects (font (size 1 1) (thickness 0.15)))
     )
-    (fp_text value EXT (at -1.27 2.54 270) (layer F.SilkS)
+    (fp_text value EXT (at 1.905 2.54 270) (layer F.SilkS)
       (effects (font (size 1 1) (thickness 0.15)))
     )
@@
       (effects (font (size 1 1) (thickness 0.15)))
     )
-    (fp_text value "Data P" (at 0 4.87 270) (layer F.SilkS)
+    (fp_text value "Data P" (at 0.635 5.08 270) (layer F.SilkS)
       (effects (font (size 1 1) (thickness 0.15)))
     )
@@
       (effects (font (size 1 1) (thickness 0.15)))
     )
-    (fp_text value PWR (at -1.905 3.175 180) (layer F.SilkS)
+    (fp_text value PWR (at 0 -3.175 180) (layer F.SilkS)
       (effects (font (size 1 1) (thickness 0.15)))
     )
@@
       (net 4 GND))
   )
-  (gr_text "12V\n\nGND" (at 134.62 73.66 180) (layer F.SilkS)
+  (gr_text "Ver 3" (at 118.11 97.155) (layer F.SilkS)
+    (effects (font (size 1.5 1.5) (thickness 0.3)))
+  )
+  (gr_text "12V\n\n\nGND" (at 134.62 73.66 180) (layer F.SilkS)
     (effects (font (size 1 1) (thickness 0.2)))
   )

Commit message: update
Routing:
- net +5V: track 16.0 -> 22.3 mm
Changed lines of the file:
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@@
   (general
     (links 40)
-    (no_connects 1)
+    (no_connects 0)
     (area 102.202857 54.27 155.607143 103.945)
     (thickness 1.6)
     (drawings 9)
-    (tracks 73)
+    (tracks 74)
     (zones 0)
     (modules 27)
@@
   (segment (start 117.475 78.74) (end 117.475 66.675) (width 0.25) (layer B.Cu) (net 2))
   (segment (start 114.935 81.28) (end 117.475 78.74) (width 0.25) (layer B.Cu) (net 2))
+  (segment (start 120.04 83.82) (end 126.34 83.82) (width 1) (layer B.Cu) (net 3))
   (segment (start 130.08 83.82) (end 126.34 83.82) (width 1) (layer B.Cu) (net 3) (status 30))
   (segment (start 120.04 83.82) (end 118.11 83.82) (width 1) (layer B.Cu) (net 3) (status 10))
