File: ax12/electrical/power-v5/_autosave-robot.kicad_pcb (KiCad board)
At the start: 2 copper layers, 49.5 x 49.5 mm, 19 parts, among them J1 C1-2, J10 LEG2, J11 EXT, J12 LEG4, J13 EXT, J14 C3-4, J15 LEG3, J16 LEG3-4, J2 RPi, J3 Data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

Commit message: pcb updates
Parts:
- moved J2 5.46 mm to (133.3, 85.1), turned to 90 degrees
- moved J16 2.54 mm to (142.9, 64.8)
- moved R1 0.64 mm to (121.9, 102.2)
Changed lines of the file:
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@@
     (tags "LED 1206")
     (attr smd)
-    (fp_text reference D1 (at 0 1.905 180) (layer F.SilkS)
+    (fp_text reference D1 (at -4.445 0 270) (layer F.SilkS)
       (effects (font (size 1 1) (thickness 0.15)))
     )
@@
   )
   (module Resistors_SMD:R_1206_HandSoldering (layer F.Cu)
-    (at 121.92 101.6 180)
+    (at 121.92 102.235 180)
     (descr "Resistor SMD 1206, hand soldering")
     (tags "resistor 1206")
     (attr smd)
-    (fp_text reference R1 (at 2.54 -1.905 180) (layer F.SilkS)
-      (effects (font (size 1 1) (thickness 0.15)))
-    )
-    (fp_text value 2.4k (at -1.27 -1.905 180) (layer F.SilkS)
+    (fp_text reference R1 (at -4.445 0 270) (layer F.SilkS)
+      (effects (font (size 1 1) (thickness 0.15)))
+    )
+    (fp_text value 2.4k (at 0 1.905 180) (layer F.SilkS)
       (effects (font (size 1 1) (thickness 0.15)))
     )
@@
   )
   (module Connectors_Molex:Molex_SPOX-5267_22-03-5035_03x2.54mm_Straight (layer F.Cu)
-    (at 130.175 80.645)
+    (at 133.35 85.09 90)
     (descr "Connector Headers with Friction Lock, 22-03-5035, http://www.molex.com/pdm_docs/ps/PS-5264-001-001.pdf")
     (tags "connector molex SPOX 5267 22-03-5035")
-    (fp_text reference J2 (at 2.54 -3.81) (layer F.Fab)
-      (effects (font (size 1 1) (thickness 0.15)))
-    )
-    (fp_text value RPi (at 2.54 2.54) (layer F.SilkS)
+    (fp_text reference J2 (at 2.54 -3.81 90) (layer F.Fab)
+      (effects (font (size 1 1) (thickness 0.15)))
+    )
+    (fp_text value RPi (at 2.54 2.54 90) (layer F.SilkS)
       (effects (font (size 1 1) (thickness 0.15)))
     )
@@
     (fp_line (start -2.35 1.7) (end 6.35 1.7) (layer F.Fab) (width 0.1))
     (fp_line (start -2.35 -3) (end -2.35 1.7) (layer F.Fab) (width 0.1))
-    (pad 1 thru_hole rect (at 0 0) (size 2 2.6) (drill 1.2) (layers *.Cu *.Mask)
-      (net 1 DATA))
-    (pad 2 thru_hole oval (at 2.54 0) (size 2 2.6) (drill 1.2) (layers *.Cu *.Mask)
+    (pad 1 thru_hole rect (at 0 0 90) (size 2 2.6) (drill 1.2) (layers *.Cu *.Mask)
+      (net 1 DATA))
+    (pad 2 thru_hole oval (at 2.54 0 90) (size 2 2.6) (drill 1.2) (layers *.Cu *.Mask)
       (net 5 "Net-(J1-Pad2)"))
-    (pad 3 thru_hole oval (at 5.08 0) (size 2 2.6) (drill 1.2) (layers *.Cu *.Mask)
+    (pad 3 thru_hole oval (at 5.08 0 90) (size 2 2.6) (drill 1.2) (layers *.Cu *.Mask)
       (net 2 GND))
     (model ${KISYS3DMOD}/Connectors_Molex.3dshapes/Molex_SPOX-5267_22-03-5035_03x2.54mm_Straight.wrl
@@
   )
   (module TerminalBlocks_Phoenix:TerminalBlock_Phoenix_MKDS1.5-2pol (layer F.Cu)
-    (at 145.415 64.77 180)
+    (at 142.875 64.77 180)
     (descr "2-way 5mm pitch terminal block, Phoenix MKDS series")
     (fp_text reference J16 (at 2.5 5.9 180) (layer F.SilkS)
