File: ax12/electrical/power-v5/robot.kicad_pcb (KiCad board)
At the start: 2 copper layers, 49.5 x 49.5 mm, 21 parts, among them J1 C1-2, J10 LEG2, J11 EXT, J12 LEG4, J13 EXT, J14 C3-4, J15 LEG3, J2 RPi, J3 Data, J4 PWR1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

Commit message: pcb updates
Parts:
- removed J4: PWR1, Connectors_Molex:Molex_SPOX-5267_22-03-5035_03x2.54mm_Straight
- removed J5: PWR3, Connectors_Molex:Molex_SPOX-5267_22-03-5035_03x2.54mm_Straight
- removed J6: PWR2, Connectors_Molex:Molex_SPOX-5267_22-03-5035_03x2.54mm_Straight
- removed J9: PWR4, Connectors_Molex:Molex_SPOX-5267_22-03-5035_03x2.54mm_Straight
- added J16: LEG3-4, TerminalBlocks_Phoenix:TerminalBlock_Phoenix_MKDS1.5-2pol, F.Cu at (142.9, 64.8)
- added J7: LEG1-2, TerminalBlocks_Phoenix:TerminalBlock_Phoenix_MKDS1.5-2pol, F.Cu at (127.6, 64.8)
- moved REF*** 50.6 mm to (183.5, 62.9)
- moved J11 47.9 mm to (113.7, 94.6), turned to 0 degrees
- moved J14 37.3 mm to (149.2, 80.6), turned to 0 degrees
- moved J10 35.2 mm to (113.7, 88.9), turned to 0 degrees
- moved J15 27.9 mm to (149.2, 74.9), turned to 0 degrees
- moved J12 12.3 mm to (149.2, 88.3), turned to 0 degrees
- moved J8 10.6 mm to (113.7, 74.9), turned to 0 degrees
- moved J2 9.86 mm to (130.2, 80.6)
- moved J1 8.98 mm to (113.7, 80.6), turned to 0 degrees
- moved D1 7.41 mm to (121.9, 106.0), turned to 180 degrees
- moved R1 6.25 mm to (121.9, 102.2)
- moved J13 4.49 mm to (149.2, 94.0), turned to 0 degrees
- moved J3 0.63 mm to (136.5, 103.5)
Connections:
- J10 pad 2: Net-(J10-Pad2) -> Net-(J1-Pad2)
- J11 pad 2: Net-(J10-Pad2) -> Net-(J1-Pad2)
- J12 pad 2: +12V -> Net-(J12-Pad2)
- J13 pad 2: +12V -> Net-(J12-Pad2)
- J14 pad 2: Net-(J14-Pad2) -> Net-(J12-Pad2)
- J15 pad 2: Net-(J14-Pad2) -> Net-(J12-Pad2)
- J2 pad 2: +12V -> Net-(J1-Pad2)
- J3 pad 2: +12V -> Net-(J12-Pad2)

Commit message: update
Parts:
- moved J2 5.46 mm to (133.3, 85.1), turned to 90 degrees
Changed lines of the file:
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@@
   )
   (module Connectors_Molex:Molex_SPOX-5267_22-03-5035_03x2.54mm_Straight (layer F.Cu)
-    (at 130.175 80.645)
+    (at 133.35 85.09 90)
     (descr "Connector Headers with Friction Lock, 22-03-5035, http://www.molex.com/pdm_docs/ps/PS-5264-001-001.pdf")
     (tags "connector molex SPOX 5267 22-03-5035")
-    (fp_text reference J2 (at 2.54 -3.81) (layer F.Fab)
+    (fp_text reference J2 (at 2.54 -3.81 90) (layer F.Fab)
       (effects (font (size 1 1) (thickness 0.15)))
     )
-    (fp_text value RPi (at 2.54 2.54) (layer F.SilkS)
+    (fp_text value RPi (at 2.54 2.54 90) (layer F.SilkS)
       (effects (font (size 1 1) (thickness 0.15)))
     )
@@
     (fp_line (start -2.35 1.7) (end 6.35 1.7) (layer F.Fab) (width 0.1))
     (fp_line (start -2.35 -3) (end -2.35 1.7) (layer F.Fab) (width 0.1))
-    (pad 1 thru_hole rect (at 0 0) (size 2 2.6) (drill 1.2) (layers *.Cu *.Mask)
+    (pad 1 thru_hole rect (at 0 0 90) (size 2 2.6) (drill 1.2) (layers *.Cu *.Mask)
       (net 1 DATA))
-    (pad 2 thru_hole oval (at 2.54 0) (size 2 2.6) (drill 1.2) (layers *.Cu *.Mask)
+    (pad 2 thru_hole oval (at 2.54 0 90) (size 2 2.6) (drill 1.2) (layers *.Cu *.Mask)
       (net 5 "Net-(J1-Pad2)"))
-    (pad 3 thru_hole oval (at 5.08 0) (size 2 2.6) (drill 1.2) (layers *.Cu *.Mask)
+    (pad 3 thru_hole oval (at 5.08 0 90) (size 2 2.6) (drill 1.2) (layers *.Cu *.Mask)
       (net 2 GND))
     (model ${KISYS3DMOD}/Connectors_Molex.3dshapes/Molex_SPOX-5267_22-03-5035_03x2.54mm_Straight.wrl

Commit message: power version 5 done and reorg
Parts:
- added ?: , Mounting_Holes:MountingHole_2.2mm_M2, F.Cu at (132.1, 83.8)
- REF***: value OSHW-Logo2_9.8x8mm_SilkScreen -> (none)
- moved REF*** 52.2 mm to (132.7, 74.9)
- moved J2 9.55 mm to (132.7, 94.6)
- moved J13 1.91 mm to (149.2, 95.9)
- moved J7 1.90 mm to (129.5, 64.8)
- moved J10 1.27 mm to (113.7, 87.6)
- moved J11 1.27 mm to (113.7, 95.9)
- moved ? 0.64 mm to (156.2, 62.2)
- moved ? 0.64 mm to (156.2, 106.7)
- moved ? 0.64 mm to (111.8, 106.7)
- moved J1 0.64 mm to (113.7, 81.3)
- moved J12 0.64 mm to (149.2, 87.6)
- moved J14 0.64 mm to (149.2, 81.3)
Connections:
- D1 pad 2: +12V -> Net-(D1-Pad2)
- J1 pad 2: Net-(J1-Pad2) -> Net-(D1-Pad2)
- J10 pad 2: Net-(J1-Pad2) -> Net-(D1-Pad2)
- J11 pad 2: Net-(J1-Pad2) -> Net-(D1-Pad2)
- J2 pad 2: Net-(J1-Pad2) -> Net-(D1-Pad2)
- J7 pad 2: Net-(J1-Pad2) -> Net-(D1-Pad2)
- J8 pad 2: Net-(J1-Pad2) -> Net-(D1-Pad2)
Routing:
- net Net-(J12-Pad2): track 0.00 -> 140.6 mm
- net Net-(D1-Pad2): track 0.00 -> 128.9 mm, vias 0 -> 1
- net DATA: track 0.00 -> 90.3 mm
- net Net-(D1-Pad1): track 0.00 -> 3.81 mm
- added copper zone on B.Cu, net GND
- added copper zone on F.Cu, net GND
Other:
- outline, holes or cut-outs redrawn
- net class A removed
