File: ax12/electrical/power-v5/robot.sch (KiCad schematic (older format))
At the start: 16 parts, among them J1 C1-2, J10 LEG2, J11 EXT, J12 LEG4, J13 EXT, J14 C3-4, J15 LEG3, J2 RPi, J3 Data, J4 PWR1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

Commit message: pcb updates
Parts:
- removed J4: PWR1, Connectors_Molex:Molex_SPOX-5267_22-03-5035_03x2.54mm_Straight, symbol Conn_01x03
- removed J5: PWR3, Connectors_Molex:Molex_SPOX-5267_22-03-5035_03x2.54mm_Straight, symbol Conn_01x03
- removed J6: PWR2, Connectors_Molex:Molex_SPOX-5267_22-03-5035_03x2.54mm_Straight, symbol Conn_01x03
- removed J9: PWR4, Connectors_Molex:Molex_SPOX-5267_22-03-5035_03x2.54mm_Straight, symbol Conn_01x03
- added J16: LEG3-4, TerminalBlocks_Phoenix:TerminalBlock_Phoenix_MKDS1.5-2pol, symbol Screw_Terminal_01x02
- added J7: LEG1-2, TerminalBlocks_Phoenix:TerminalBlock_Phoenix_MKDS1.5-2pol, symbol Screw_Terminal_01x02
Connections:
- net +12V: no longer J12.2 (Pin_2), J13.2 (Pin_2), J2.2 (Pin_2), J3.2 (Pin_2)
- net GND: now also J16.1 (Pin_1), J7.1 (Pin_1)
- net at J1.2 (Pin_2), J8.2 (Pin_2): now also J10.2 (Pin_2), J11.2 (Pin_2), J2.2 (Pin_2), J7.2 (Pin_2)
- net at J14.2 (Pin_2), J15.2 (Pin_2): now also J12.2 (Pin_2), J13.2 (Pin_2), J3.2 (Pin_2), J16.2 (Pin_2)
- no-connect marks 4 -> 0
Other:
- moved on the sheet: D1, J10, J11, J12, J13, J14, J15, J2, J3, R1

Commit message: power version 5 done and reorg
Connections:
- net +12V: no longer D1.2 (A)
- net at J1.2 (Pin_2), J10.2 (Pin_2), J11.2 (Pin_2)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: now also D1.2 (A)
Other:
- note added: "AX-12A Quadruped Power Distribution Board\nVersion 5\nNote: the molex pin numbers appear to be in reverse\n--------------------------------\n1 - Data\n2 - 12V\n3 - Ground\n----------------------------\nTrying to keep the current draw around 3A per cable:\nCX-Y: coxa motors for leg X and leg Y\nLegX: tibia, fibia, and tarsus motors for leg X"
- note added: "Data and Power Alternate Interfaces"
- note removed: "AX-12A Quadruped Power Distribution Board\nVersion 5\nNote: the molex pin numbers appear to be in reverse\n--------------------------------\n1 - Data\n2 - 12V\n3 - Ground"
- note removed: "Data and Alternate Interfaces"
- moved on the sheet: D1, R1
Changed lines of the file:
@@
 L LED D1
 U 1 1 5ACD24C2
-P 4550 2550
-F 0 "D1" H 4550 2650 50  0000 C CNN
-F 1 "PWR" H 4550 2450 50  0000 C CNN
-F 2 "LEDs:LED_1206_HandSoldering" H 4550 2550 50  0001 C CNN
-F 3 "" H 4550 2550 50  0001 C CNN
-	1    4550 2550
+P 5850 2850
+F 0 "D1" H 5850 2950 50  0000 C CNN
+F 1 "PWR" H 5850 2750 50  0000 C CNN
+F 2 "LEDs:LED_1206_HandSoldering" H 5850 2850 50  0001 C CNN
+F 3 "" H 5850 2850 50  0001 C CNN
+	1    5850 2850
 	0    -1   -1   0
 $EndComp
@@
 L R R1
 U 1 1 5ACD2583
-P 4550 3000
-F 0 "R1" V 4630 3000 50  0000 C CNN
-F 1 "2.4k" V 4550 3000 50  0000 C CNN
-F 2 "Resistors_SMD:R_1206_HandSoldering" V 4480 3000 50  0001 C CNN
-F 3 "" H 4550 3000 50  0001 C CNN
-	1    4550 3000
-	1    0    0    -1
-$EndComp
-$Comp
-L +12V #PWR05
-U 1 1 5ACD2665
-P 4550 2300
-F 0 "#PWR05" H 4550 2150 50  0001 C CNN
-F 1 "+12V" H 4550 2440 50  0000 C CNN
-F 2 "" H 4550 2300 50  0001 C CNN
-F 3 "" H 4550 2300 50  0001 C CNN
-	1    4550 2300
+P 5850 3300
+F 0 "R1" V 5930 3300 50  0000 C CNN
+F 1 "2.4k" V 5850 3300 50  0000 C CNN
+F 2 "Resistors_SMD:R_1206_HandSoldering" V 5780 3300 50  0001 C CNN
+F 3 "" H 5850 3300 50  0001 C CNN
+	1    5850 3300
 	1    0    0    -1
 $EndComp
@@
 L GND #PWR06
 U 1 1 5ACD2691
-P 4550 3300
-F 0 "#PWR06" H 4550 3050 50  0001 C CNN
-F 1 "GND" H 4550 3150 50  0000 C CNN
-F 2 "" H 4550 3300 50  0001 C CNN
-F 3 "" H 4550 3300 50  0001 C CNN
-	1    4550 3300
-	1    0    0    -1
-$EndComp
-Wire Wire Line
-	4550 2300 4550 2400
-Wire Wire Line
-	4550 2700 4550 2850
-Wire Wire Line
-	4550 3150 4550 3300
+P 5850 3600
+F 0 "#PWR06" H 5850 3350 50  0001 C CNN
+F 1 "GND" H 5850 3450 50  0000 C CNN
+F 2 "" H 5850 3600 50  0001 C CNN
+F 3 "" H 5850 3600 50  0001 C CNN
+	1    5850 3600
+	1    0    0    -1
+$EndComp
+Wire Wire Line
+	5850 2200 5850 2700
+Wire Wire Line
+	5850 3000 5850 3150
+Wire Wire Line
+	5850 3450 5850 3600
 $Comp
 L Conn_01x03 J14
@@
 	9350 3650 9000 3650
 Connection ~ 9000 3650
-Text Notes 4400 1350 0    60   ~ 0
-AX-12A Quadruped Power Distribution Board\nVersion 5\nNote: the molex pin numbers appear to be in reverse\n--------------------------------\n1 - Data\n2 - 12V\n3 - Ground
+Text Notes 4400 1600 0    60   ~ 0
+AX-12A Quadruped Power Distribution Board\nVersion 5\nNote: the molex pin numbers appear to be in reverse\n--------------------------------\n1 - Data\n2 - 12V\n3 - Ground\n----------------------------\nTrying to keep the current draw around 3A per cable:\nCX-Y: coxa motors for leg X and leg Y\nLegX: tibia, fibia, and tarsus motors for leg X
 Text Notes 4350 1950 0    60   ~ 0
 Power LED
@@
 AX-12A Interfaces
 Text Notes 7400 5300 0    60   ~ 0
-Data and Alternate Interfaces
+Data and Power Alternate Interfaces
 $Comp
 L Conn_01x03 J2
@@
 Wire Notes Line
 	6000 5550 6000 4350
+Wire Wire Line
+	5850 2200 6650 2200
+Wire Wire Line
+	6650 2200 6650 2400
+Connection ~ 6650 2400
 $EndSCHEMATC
