File: ax12/electrical/rpi/robot.sch (KiCad schematic (older format))
At the start: 30 parts, among them J1 12V, J2 LEG1, J3 Pi USB Pwr, J4 Serial, J5 LEG2, J6 LEG3, J7 LEG4, J8 Data P, J9 Data S, U1 LM317_12, U2 AP1117-50, U3 74LS126, U4 LM317_34

Commit message: update
Parts:
- removed C3, C4: .1, Capacitors_THT:CP_Radial_D6.3mm_P2.50mm, symbol CP
- removed C5, C6: C, Capacitors_SMD:C_1206_HandSoldering, symbol C
- removed J1: 12V, TerminalBlocks_Phoenix:TerminalBlock_Phoenix_PT-3.5mm_2pol, symbol Screw_Terminal_01x02
- removed J2: LEG1, Connectors_Molex:Molex_MicroLatch-53253-0370_03x2.00mm_Straight, symbol Conn_01x03
- removed J5: LEG2, Connectors_Molex:Molex_MicroLatch-53253-0370_03x2.00mm_Straight, symbol Conn_01x03
- removed J6: LEG3, Connectors_Molex:Molex_MicroLatch-53253-0370_03x2.00mm_Straight, symbol Conn_01x03
- removed J7: LEG4, Connectors_Molex:Molex_MicroLatch-53253-0370_03x2.00mm_Straight, symbol Conn_01x03
- removed J8: Data P, Pin_Headers:Pin_Header_Straight_1x03_Pitch2.54mm, symbol Conn_01x03
- removed R1, R3: 330, Resistors_SMD:R_1206_HandSoldering, symbol R
- removed R2, R4: 1.8k, Resistors_SMD:R_1206_HandSoldering, symbol R
- removed U1: LM317_12, TO_SOT_Packages_THT:TO-220-3_Horizontal, symbol LM317_TO3
- removed U4: LM317_34, TO_SOT_Packages_THT:TO-220-3_Horizontal, symbol LM317_TO3
- added J1: Raspberry_Pi_2_3, Pin_Headers:Pin_Header_Straight_2x20_Pitch2.54mm, symbol Raspberry_Pi_2_3
- added J2: IMU, Pin_Headers:Pin_Header_Straight_1x04_Pitch2.54mm, symbol Conn_01x04
- added J3: Lidar, Pin_Headers:Pin_Header_Straight_1x04_Pitch2.54mm, symbol Conn_01x04
- added J7: Audio, Pin_Headers:Pin_Header_Straight_1x05_Pitch2.54mm, symbol Conn_01x05
- D2: renamed from D1; footprint LEDs:LED_D5.0mm -> LEDs:LED_1206_HandSoldering
- D3: renamed from D2; footprint LEDs:LED_D5.0mm -> LEDs:LED_1206_HandSoldering
- renumbered D3 to D1, J9 to J5, J3 to J6, R8 to R1, R5 to R2, R6 to R3, R7 to R4, U2 to U1, U3 to U2
Connections:
- net labels removed: +5VA, DATA, GNDA, PWR12, PWR34
- wire segments 108 -> 86
Other:
- note removed: "Power System and Servo Bus Interface"

Commit message: jst library
Parts:
- removed D2: TX, LEDs:LED_1206_HandSoldering, symbol LED
- removed D3: RX, LEDs:LED_1206_HandSoldering, symbol LED
- removed J5: Data S, Pin_Headers:Pin_Header_Straight_1x03_Pitch2.54mm, symbol Conn_01x03
- removed R2: 10k, Resistors_SMD:R_1206_HandSoldering, symbol R
- removed R3, R4: 330, Resistors_SMD:R_1206_HandSoldering, symbol R
- removed U2: 74LS126, Housings_SOIC:SOIC-14_3.9x8.7mm_Pitch1.27mm, symbol 74LS126
- added J5: AN, Pin_Headers:Pin_Header_Straight_1x02_Pitch2.54mm, symbol Conn_01x08
- added U2: MCP3208, symbol MCP3208
- J2: symbol Conn_01x04 -> Conn_01x06
- J4: value Serial -> I2C
- J7: symbol Conn_01x05 -> Conn_01x07
Connections:
- net labels added: +3V3, BCLK, CS, DIN, IMU-RST, LRC, MISO, MOSI, SPI-CLK
- net labels removed: DTR, RXO, TXI
- no-connect marks 3 -> 5
Other:
- note added: "5V\nGnd\nSD\nGAIN\nDIN\nBCLK\nLRC"
- note added: "These are board pins"
- note added: "Vin\n3Vo\nGND\nSCL\nSDA\nRST"
- note removed: "DATA"

Commit message: up
Parts:
- removed J5: AN, Pin_Headers:Pin_Header_Straight_1x02_Pitch2.54mm, symbol Conn_01x08
- removed U2: MCP3208, symbol MCP3208
- added J?: SPI, Pin_Headers:Pin_Header_Straight_1x04_Pitch2.54mm, symbol Conn_01x06
Connections:
- wire segments 86 -> 77
Other:
- moved on the sheet: J4
Changed lines of the file:
@@
 L Conn_01x04 J4
 U 1 1 5AA1A6A1
-P 5700 2050
-F 0 "J4" H 5700 2250 50  0000 C CNN
-F 1 "I2C" H 5700 1750 50  0000 C CNN
-F 2 "Pin_Headers:Pin_Header_Straight_1x04_Pitch2.54mm" H 5700 2050 50  0001 C CNN
-F 3 "" H 5700 2050 50  0001 C CNN
-	1    5700 2050
+P 5800 1950
+F 0 "J4" H 5800 2150 50  0000 C CNN
+F 1 "I2C" H 5800 1650 50  0000 C CNN
+F 2 "Pin_Headers:Pin_Header_Straight_1x04_Pitch2.54mm" H 5800 1950 50  0001 C CNN
+F 3 "" H 5800 1950 50  0001 C CNN
+	1    5800 1950
 	1    0    0    -1
 $EndComp
@@
 	3700 1650 3700 1500
 Wire Wire Line
-	4400 2050 5500 2050
-Wire Wire Line
-	4400 2150 5500 2150
+	4400 2050 5600 2050
+Wire Wire Line
+	4400 2150 5600 2150
 Wire Wire Line
 	3100 4250 3100 4400
@@
 L GND #PWR017
 U 1 1 5AA1A931
-P 5400 2350
-F 0 "#PWR017" H 5400 2100 50  0001 C CNN
-F 1 "GND" H 5400 2200 50  0000 C CNN
-F 2 "" H 5400 2350 50  0001 C CNN
-F 3 "" H 5400 2350 50  0001 C CNN
-	1    5400 2350
+P 5300 1850
+F 0 "#PWR017" H 5300 1600 50  0001 C CNN
+F 1 "GND" H 5300 1700 50  0000 C CNN
+F 2 "" H 5300 1850 50  0001 C CNN
+F 3 "" H 5300 1850 50  0001 C CNN
+	1    5300 1850
 	1    0    0    -1
 $EndComp
@@
 L +3V3 #PWR020
 U 1 1 5AA1B009
-P 5400 1900
-F 0 "#PWR020" H 5400 1750 50  0001 C CNN
-F 1 "+3V3" H 5400 2040 50  0000 C CNN
-F 2 "" H 5400 1900 50  0001 C CNN
-F 3 "" H 5400 1900 50  0001 C CNN
-	1    5400 1900
-	1    0    0    -1
-$EndComp
-Wire Wire Line
-	5500 2250 5400 2250
-Wire Wire Line
-	5400 2250 5400 2350
-Wire Wire Line
-	5500 1950 5400 1950
-Wire Wire Line
-	5400 1950 5400 1900
+P 5500 1750
+F 0 "#PWR020" H 5500 1600 50  0001 C CNN
+F 1 "+3V3" H 5500 1890 50  0000 C CNN
+F 2 "" H 5500 1750 50  0001 C CNN
+F 3 "" H 5500 1750 50  0001 C CNN
+	1    5500 1750
+	1    0    0    -1
+$EndComp
+Wire Wire Line
+	5500 1850 5500 1750
 Text Notes 5300 900  1    60   ~ 0
 Vin\n3Vo\nGND\nSCL\nSDA\nRST
@@
 Wire Wire Line
 	5300 1300 5500 1300
-$Comp
-L MCP3208 U2
-U 1 1 5AA1C03D
-P 8800 1800
-F 0 "U2" H 8600 2325 50  0000 R CNN
-F 1 "MCP3208" H 8600 2250 50  0000 R CNN
-F 2 "" H 8900 1900 50  0001 C CNN
-F 3 "" H 8900 1900 50  0001 C CNN
-	1    8800 1800
-	-1   0    0    1
-$EndComp
 Text GLabel 4600 2850 2    60   Output ~ 0
 CS
@@
 SPI-CLK
 Wire Wire Line
-	7900 1600 8200 1600
-Wire Wire Line
-	7900 1700 8200 1700
-Wire Wire Line
-	7900 1800 8200 1800
-Wire Wire Line
-	7900 1900 8200 1900
-Wire Wire Line
 	4400 2850 4600 2850
 Wire Wire Line
@@
 	4400 3150 4600 3150
 $Comp
-L +3V3 #PWR021
-U 1 1 5AA1CE62
-P 8350 2550
-F 0 "#PWR021" H 8350 2400 50  0001 C CNN
-F 1 "+3V3" H 8350 2690 50  0000 C CNN
-F 2 "" H 8350 2550 50  0001 C CNN
-F 3 "" H 8350 2550 50  0001 C CNN
-	1    8350 2550
-	1    0    0    -1
-$EndComp
-$Comp
-L GND #PWR022
-U 1 1 5AA1CE91
-P 8350 1000
-F 0 "#PWR022" H 8350 750 50  0001 C CNN
-F 1 "GND" H 8350 850 50  0000 C CNN
-F 2 "" H 8350 1000 50  0001 C CNN
-F 3 "" H 8350 1000 50  0001 C CNN
-	1    8350 1000
-	1    0    0    -1
-$EndComp
-Wire Wire Line
-	8900 1200 8900 1000
-Wire Wire Line
-	8900 1000 8350 1000
-Wire Wire Line
-	8600 1200 8600 1000
-Connection ~ 8600 1000
-Wire Wire Line
-	8350 2550 8900 2550
-Wire Wire Line
-	8600 2550 8600 2300
-Wire Wire Line
-	8900 2550 8900 2300
-Connection ~ 8600 2550
-$Comp
-L Conn_01x08 J5
-U 1 1 5AA1D08A
-P 9750 1800
-F 0 "J5" H 9750 2200 50  0000 C CNN
-F 1 "AN" V 9850 1800 50  0000 C CNN
-F 2 "Pin_Headers:Pin_Header_Straight_1x02_Pitch2.54mm" H 9750 1800 50  0001 C CNN
-F 3 "" H 9750 1800 50  0001 C CNN
-	1    9750 1800
-	1    0    0    1
-$EndComp
-Wire Wire Line
-	9400 1400 9550 1400
-Wire Wire Line
-	9400 1500 9550 1500
-Wire Wire Line
-	9400 1600 9550 1600
-Wire Wire Line
-	9400 1700 9550 1700
-Wire Wire Line
-	9400 1800 9550 1800
-Wire Wire Line
-	9400 1900 9550 1900
-Wire Wire Line
-	9400 2000 9550 2000
-Wire Wire Line
-	9400 2100 9550 2100
+L Conn_01x06 J?
+U 1 1 5AA22432
+P 8250 1600
+F 0 "J?" H 8250 1900 50  0000 C CNN
+F 1 "SPI" H 8250 1200 50  0000 C CNN
+F 2 "Pin_Headers:Pin_Header_Straight_1x04_Pitch2.54mm" H 8250 1600 50  0001 C CNN
+F 3 "" H 8250 1600 50  0001 C CNN
+	1    8250 1600
+	1    0    0    -1
+$EndComp
+Wire Wire Line
+	5500 1850 5600 1850
+Wire Wire Line
+	5300 1850 5300 1800
+Wire Wire Line
+	5300 1800 5400 1800
+Wire Wire Line
+	5400 1800 5400 1950
+Wire Wire Line
+	5400 1950 5600 1950
+$Comp
+L +3V3 #PWR?
+U 1 1 5AA22A0F
+P 7900 1200
+F 0 "#PWR?" H 7900 1050 50  0001 C CNN
+F 1 "+3V3" H 7900 1340 50  0000 C CNN
+F 2 "" H 7900 1200 50  0001 C CNN
+F 3 "" H 7900 1200 50  0001 C CNN
+	1    7900 1200
+	1    0    0    -1
+$EndComp
+$Comp
+L GND #PWR?
+U 1 1 5AA22A3E
+P 7450 1500
+F 0 "#PWR?" H 7450 1250 50  0001 C CNN
+F 1 "GND" H 7450 1350 50  0000 C CNN
+F 2 "" H 7450 1500 50  0001 C CNN
+F 3 "" H 7450 1500 50  0001 C CNN
+	1    7450 1500
+	1    0    0    -1
+$EndComp
+Wire Wire Line
+	8050 1500 7450 1500
+Wire Wire Line
+	8050 1400 7900 1400
+Wire Wire Line
+	7900 1400 7900 1200
+Wire Wire Line
+	8050 1900 7900 1900
+Wire Wire Line
+	8050 1800 7900 1800
+Wire Wire Line
+	8050 1700 7900 1700
+Wire Wire Line
+	8050 1600 7900 1600
 $EndSCHEMATC

Commit message: electrical update
Parts:
- added D2: TX, LEDs:LED_1206_HandSoldering, symbol LED
- added D3: RX, LEDs:LED_1206_HandSoldering, symbol LED
- added J8: SERIAL, Pin_Headers:Pin_Header_Straight_1x06_Pitch2.54mm, symbol Conn_01x06
- added J9: PWR BOARD, Pin_Headers:Pin_Header_Straight_1x03_Pitch2.54mm, symbol Conn_01x03
- added Q1: BSS138, TO_SOT_Packages_SMD:SOT-23, symbol BSS138
- added R2, R3, R4, R5: 330, Resistors_SMD:R_1206_HandSoldering, symbol R
- added U2: 74LVC1G125, TO_SOT_Packages_SMD:SOT-23-5_HandSoldering, symbol 74LVC1G125
- added U3: 74LVC1G126, TO_SOT_Packages_SMD:SOT-23-5_HandSoldering, symbol 74LVC1G126
- J2: footprint Pin_Headers:Pin_Header_Straight_1x04_Pitch2.54mm -> Pin_Headers:Pin_Header_Straight_1x06_Pitch2.54mm
- J5: renamed from J?; footprint Pin_Headers:Pin_Header_Straight_1x04_Pitch2.54mm -> Pin_Headers:Pin_Header_Straight_1x06_Pitch2.54mm
- J7: footprint Pin_Headers:Pin_Header_Straight_1x05_Pitch2.54mm -> Pin_Headers:Pin_Header_Straight_1x07_Pitch2.54mm
Connections:
- net +12V: now also J9.2 (Pin_2)
- net +3V3: now also D2.2 (A), Q1.1 (G), R3.1, U2.5 (VCC), U3.5 (VCC); no longer J1.17 (3V3)
- net +5V: now also R2.1
- net GND: now also J8.1 (Pin_1), J9.3 (Pin_3), R5.2, U2.3 (GND), U3.3 (GND)
- net MISO: no longer J5.5 (Pin_5)
- net MOSI: now also J5.5 (Pin_5)
- new net: D2.1 (K), R4.1
- new net: D3.1 (K), R5.1
- new net DATA: J9.1 (Pin_1), Q1.3 (D), R2.2
- new net DTR: J8.6 (Pin_6), Q1.2 (S), R3.2, U2.1, U2.4, U3.1, U3.2
- new net RXI: D3.2 (A), J8.5 (Pin_5), U3.4
- new net TXO: J8.4 (Pin_4), R4.2, U2.2
- no-connect marks 5 -> 24
Other:
- note added: "GND\nCTS\n3V3\nTXO\nRXI\nDTR"
- note added: "Pins: Pi (BCM)"
- note added: "Power: 5V@1.5A"
- note added: "Robotis AX-12A Servo Data to Serial Converter"
- note removed: "These are board pins"
- note removed: "XL-320 Servo Data to Serial Converter"
- moved on the sheet: J5, J7

Commit message: power 3 done :tada: :electric_plug:
Parts:
- removed Q1: BSS138, TO_SOT_Packages_SMD:SOT-23, symbol BSS138
- added Q?: BSS138, TO_SOT_Packages_SMD:SOT-23, symbol BSS138
- J8: value SERIAL -> SERIAL 3V3
- R2, R3: value 330 -> 10k
Connections:
- net +3V3: now also Q?.1 (G)
- net +5V: now also J1.4 (5V)
- net DATA: now also Q?.3 (D)
- net DTR: now also Q?.2 (S)
- no-connect marks 24 -> 23
Other:
- moved on the sheet: R2, R3
Changed lines of the file:
@@
 $EndComp
 NoConn ~ 3300 1650
-NoConn ~ 3400 1650
 $Comp
 L +3V3 #PWR016
@@
 P 9300 5050
 F 0 "U3" H 9200 5200 50  0000 C CNN
-F 1 "74LVC1G126" H 9300 4900 50  0000 C CNN
+F 1 "74LVC1G126" H 9150 4900 50  0000 C CNN
 F 2 "TO_SOT_Packages_SMD:SOT-23-5_HandSoldering" H 9300 5050 50  0001 C CNN
 F 3 "" H 9300 5050 50  0001 C CNN
@@
 $EndComp
 $Comp
-L BSS138 Q1
-U 1 1 5AA2CE83
-P 8550 4650
-F 0 "Q1" H 8750 4725 50  0000 L CNN
-F 1 "BSS138" H 8750 4650 50  0000 L CNN
-F 2 "TO_SOT_Packages_SMD:SOT-23" H 8750 4575 50  0001 L CIN
-F 3 "" H 8550 4650 50  0001 L CNN
-	1    8550 4650
-	0    -1   1    0
-$EndComp
-$Comp
 L R R3
 U 1 1 5AA2CFAD
-P 8850 4500
-F 0 "R3" V 8930 4500 50  0000 C CNN
-F 1 "330" V 8850 4500 50  0000 C CNN
-F 2 "Resistors_SMD:R_1206_HandSoldering" V 8780 4500 50  0001 C CNN
-F 3 "" H 8850 4500 50  0001 C CNN
-	1    8850 4500
+P 7800 4150
+F 0 "R3" V 7880 4150 50  0000 C CNN
+F 1 "10k" V 7800 4150 50  0000 C CNN
+F 2 "Resistors_SMD:R_1206_HandSoldering" V 7730 4150 50  0001 C CNN
+F 3 "" H 7800 4150 50  0001 C CNN
+	1    7800 4150
 	1    0    0    -1
 $EndComp
@@
 L R R2
 U 1 1 5AA2CFFB
-P 8250 4500
-F 0 "R2" V 8330 4500 50  0000 C CNN
-F 1 "330" V 8250 4500 50  0000 C CNN
-F 2 "Resistors_SMD:R_1206_HandSoldering" V 8180 4500 50  0001 C CNN
-F 3 "" H 8250 4500 50  0001 C CNN
-	1    8250 4500
+P 8450 4150
+F 0 "R2" V 8530 4150 50  0000 C CNN
+F 1 "10k" V 8450 4150 50  0000 C CNN
+F 2 "Resistors_SMD:R_1206_HandSoldering" V 8380 4150 50  0001 C CNN
+F 3 "" H 8450 4150 50  0001 C CNN
+	1    8450 4150
 	1    0    0    -1
 $EndComp
@@
 L +5V #PWR021
 U 1 1 5AA2D056
-P 8250 4250
-F 0 "#PWR021" H 8250 4100 50  0001 C CNN
-F 1 "+5V" H 8250 4390 50  0000 C CNN
-F 2 "" H 8250 4250 50  0001 C CNN
-F 3 "" H 8250 4250 50  0001 C CNN
-	1    8250 4250
+P 8450 3850
+F 0 "#PWR021" H 8450 3700 50  0001 C CNN
+F 1 "+5V" H 8450 3990 50  0000 C CNN
+F 2 "" H 8450 3850 50  0001 C CNN
+F 3 "" H 8450 3850 50  0001 C CNN
+	1    8450 3850
 	1    0    0    -1
 $EndComp
@@
 L +3V3 #PWR022
 U 1 1 5AA2DAAC
-P 8850 4250
-F 0 "#PWR022" H 8850 4100 50  0001 C CNN
-F 1 "+3V3" H 8850 4390 50  0000 C CNN
-F 2 "" H 8850 4250 50  0001 C CNN
-F 3 "" H 8850 4250 50  0001 C CNN
-	1    8850 4250
-	1    0    0    -1
-$EndComp
-Text GLabel 8100 4750 0    60   BiDi ~ 0
+P 7800 3850
+F 0 "#PWR022" H 7800 3700 50  0001 C CNN
+F 1 "+3V3" H 7800 3990 50  0000 C CNN
+F 2 "" H 7800 3850 50  0001 C CNN
+F 3 "" H 7800 3850 50  0001 C CNN
+	1    7800 3850
+	1    0    0    -1
+$EndComp
+Text GLabel 8550 4400 2    60   BiDi ~ 0
 DATA
 Text GLabel 9750 4450 2    60   Input ~ 0
@@
 P 10100 1600
 F 0 "J8" H 10100 1900 50  0000 C CNN
-F 1 "SERIAL" H 10100 1200 50  0000 C CNN
+F 1 "SERIAL 3V3" H 10100 1200 50  0000 C CNN
 F 2 "Pin_Headers:Pin_Header_Straight_1x06_Pitch2.54mm" H 10100 1600 50  0001 C CNN
 F 3 "" H 10100 1600 50  0001 C CNN
@@
 	9600 4450 9750 4450
 Wire Wire Line
-	8750 4750 9750 4750
-Wire Wire Line
 	9300 4650 9300 4850
 Connection ~ 9300 4750
 Wire Wire Line
-	8850 4650 8850 4750
-Connection ~ 8850 4750
-Wire Wire Line
-	8850 4250 8850 4350
-Wire Wire Line
-	8250 4250 8250 4350
-Wire Wire Line
-	8100 4750 8350 4750
-Wire Wire Line
 	9050 4450 9000 4450
 Wire Wire Line
@@
 Wire Wire Line
 	9550 5050 9750 5050
-Wire Wire Line
-	8250 4650 8250 4750
-Connection ~ 8250 4750
-Wire Wire Line
-	8550 4450 8550 4300
-Wire Wire Line
-	8550 4300 8850 4300
-Connection ~ 8850 4300
 Wire Wire Line
 	3100 6950 3100 7150
@@
 Text Notes 5800 3700 0    60   ~ 0
 Power: 5V@1.5A
+$Comp
+L BSS138 Q?
+U 1 1 5AAD3B03
+P 8150 4300
+F 0 "Q?" V 8400 4300 50  0000 L CNN
+F 1 "BSS138" V 8500 4150 50  0000 L CNN
+F 2 "TO_SOT_Packages_SMD:SOT-23" H 8350 4225 50  0001 L CIN
+F 3 "" H 8150 4300 50  0001 L CNN
+	1    8150 4300
+	0    1    1    0
+$EndComp
+Wire Wire Line
+	8350 4400 8550 4400
+Wire Wire Line
+	8450 4300 8450 4400
+Connection ~ 8450 4400
+Wire Wire Line
+	8450 4000 8450 3850
+Wire Wire Line
+	7800 4000 7800 3850
+Wire Wire Line
+	8150 4100 8150 3900
+Wire Wire Line
+	8150 3900 7800 3900
+Connection ~ 7800 3900
+Wire Wire Line
+	7800 4300 7800 4750
+Wire Wire Line
+	7800 4400 7950 4400
+Wire Wire Line
+	7800 4750 9750 4750
+Connection ~ 7800 4400
+$Comp
+L +5V #PWR?
+U 1 1 5AAD5DA7
+P 3400 1350
+F 0 "#PWR?" H 3400 1200 50  0001 C CNN
+F 1 "+5V" H 3400 1490 50  0000 C CNN
+F 2 "" H 3400 1350 50  0001 C CNN
+F 3 "" H 3400 1350 50  0001 C CNN
+	1    3400 1350
+	1    0    0    -1
+$EndComp
+Wire Wire Line
+	3400 1650 3400 1350
 $EndSCHEMATC

Commit message: update
Parts:
- removed C1, C2: C, Capacitors_SMD:C_1206_HandSoldering, symbol C
- removed D1: PWR, LEDs:LED_1206_HandSoldering, symbol LED
- removed J6: Pi USB Pwr, Pin_Headers:Pin_Header_Straight_1x02_Pitch2.54mm, symbol Conn_01x02
- removed R1: 330, Resistors_SMD:R_1206_HandSoldering, symbol R
- removed U1: AP1117-50, TO_SOT_Packages_SMD:SOT-223-3_TabPin2, symbol AP1117-50
- J3: value Lidar -> serial0
- J5: value SPI -> SPI 3V3
- J8: value SERIAL 3V3 -> USB SER 3V3
- J9: value PWR BOARD -> DATA 5V; footprint Pin_Headers:Pin_Header_Straight_1x03_Pitch2.54mm -> Pin_Headers:Pin_Header_Straight_1x02_Pitch2.54mm; symbol Conn_01x03 -> Conn_01x02
- gave numbers to parts that had none: 1
Connections:
- net +12V is gone; now on net GND: J9.2 (Pin_2)
- net +3V3: no longer D2.2 (A), Q1.1 (G), R3.1, U2.5 (VCC), U3.5 (VCC)
- net +5V: now also J1.2 (5V)
- net DTR: no longer Q1.2 (S), R3.2, U2.4, U3.2
- net GND: no longer J9.3 (Pin_3)
- net VCC: now reaches J1.17 (3V3)
- net VCC: now also D2.2 (A), Q1.1 (G), R3.1, U2.5 (VCC), U3.5 (VCC)
- new net: Q1.2 (S), R3.2, U2.4, U3.2
- no-connect marks 23 -> 21
Other:
- note removed: "Power: 5V@1.5A"

Commit message: power version 5 done and reorg
Parts:
- removed D2: TX, LEDs:LED_1206_HandSoldering, symbol LED
- removed D3: RX, LEDs:LED_1206_HandSoldering, symbol LED
- removed R4, R5: 330, Resistors_SMD:R_1206_HandSoldering, symbol R
Other:
- moved on the sheet: J5
Changed lines of the file:
@@
 Text GLabel 4600 2850 2    60   Output ~ 0
 CS
-Text GLabel 8550 1400 0    60   Output ~ 0
+Text GLabel 8200 1350 0    60   Output ~ 0
 CS
 Text GLabel 4600 3050 2    60   Output ~ 0
@@
 Text GLabel 4600 2950 2    60   Output ~ 0
 MISO
-Text GLabel 8550 1600 0    60   Output ~ 0
+Text GLabel 8200 1550 0    60   Output ~ 0
 MOSI
-Text GLabel 8550 1500 0    60   Output ~ 0
+Text GLabel 8200 1450 0    60   Output ~ 0
 MISO
 Text GLabel 4600 3150 2    60   Output ~ 0
 SPI-CLK
-Text GLabel 8550 1700 0    60   Output ~ 0
+Text GLabel 8200 1650 0    60   Output ~ 0
 SPI-CLK
 $Comp
 L Conn_01x06 J5
 U 1 1 5AA22432
-P 8900 1400
-F 0 "J5" H 8900 1700 50  0000 C CNN
-F 1 "SPI 3V3" H 8900 1000 50  0000 C CNN
-F 2 "Pin_Headers:Pin_Header_Straight_1x06_Pitch2.54mm" H 8900 1400 50  0001 C CNN
-F 3 "" H 8900 1400 50  0001 C CNN
-	1    8900 1400
+P 8550 1350
+F 0 "J5" H 8550 1650 50  0000 C CNN
+F 1 "SPI 3V3" H 8550 950 50  0000 C CNN
+F 2 "Pin_Headers:Pin_Header_Straight_1x06_Pitch2.54mm" H 8550 1350 50  0001 C CNN
+F 3 "" H 8550 1350 50  0001 C CNN
+	1    8550 1350
 	1    0    0    -1
 $EndComp
@@
 L +3V3 #PWR013
 U 1 1 5AA22A0F
-P 8550 1000
-F 0 "#PWR013" H 8550 850 50  0001 C CNN
-F 1 "+3V3" H 8550 1140 50  0000 C CNN
-F 2 "" H 8550 1000 50  0001 C CNN
-F 3 "" H 8550 1000 50  0001 C CNN
-	1    8550 1000
+P 8200 950
+F 0 "#PWR013" H 8200 800 50  0001 C CNN
+F 1 "+3V3" H 8200 1090 50  0000 C CNN
+F 2 "" H 8200 950 50  0001 C CNN
+F 3 "" H 8200 950 50  0001 C CNN
+	1    8200 950
 	1    0    0    -1
 $EndComp
@@
 L GND #PWR014
 U 1 1 5AA22A3E
-P 8100 1300
-F 0 "#PWR014" H 8100 1050 50  0001 C CNN
-F 1 "GND" H 8100 1150 50  0000 C CNN
-F 2 "" H 8100 1300 50  0001 C CNN
-F 3 "" H 8100 1300 50  0001 C CNN
-	1    8100 1300
+P 7750 1250
+F 0 "#PWR014" H 7750 1000 50  0001 C CNN
+F 1 "GND" H 7750 1100 50  0000 C CNN
+F 2 "" H 7750 1250 50  0001 C CNN
+F 3 "" H 7750 1250 50  0001 C CNN
+	1    7750 1250
 	1    0    0    -1
 $EndComp
@@
 $EndComp
 $Comp
-L LED D2
-U 1 1 5AA2F8B2
-P 9650 3850
-F 0 "D2" H 9650 3950 50  0000 C CNN
-F 1 "TX" H 9650 3750 50  0000 C CNN
-F 2 "LEDs:LED_1206_HandSoldering" H 9650 3850 50  0001 C CNN
-F 3 "" H 9650 3850 50  0001 C CNN
-	1    9650 3850
-	0    -1   -1   0
-$EndComp
-$Comp
-L LED D3
-U 1 1 5AA2F96E
-P 9650 5250
-F 0 "D3" H 9650 5350 50  0000 C CNN
-F 1 "RX" H 9650 5150 50  0000 C CNN
-F 2 "LEDs:LED_1206_HandSoldering" H 9650 5250 50  0001 C CNN
-F 3 "" H 9650 5250 50  0001 C CNN
-	1    9650 5250
-	0    -1   -1   0
-$EndComp
-$Comp
-L R R4
-U 1 1 5AA2FA9D
-P 9650 4250
-F 0 "R4" V 9730 4250 50  0000 C CNN
-F 1 "330" V 9650 4250 50  0000 C CNN
-F 2 "Resistors_SMD:R_1206_HandSoldering" V 9580 4250 50  0001 C CNN
-F 3 "" H 9650 4250 50  0001 C CNN
-	1    9650 4250
-	1    0    0    -1
-$EndComp
-$Comp
-L R R5
-U 1 1 5AA2FB65
-P 9650 5650
-F 0 "R5" V 9730 5650 50  0000 C CNN
-F 1 "330" V 9650 5650 50  0000 C CNN
-F 2 "Resistors_SMD:R_1206_HandSoldering" V 9580 5650 50  0001 C CNN
-F 3 "" H 9650 5650 50  0001 C CNN
-	1    9650 5650
-	1    0    0    -1
-$EndComp
-$Comp
-L GND #PWR020
-U 1 1 5AA2FDB7
-P 9650 5900
-F 0 "#PWR020" H 9650 5650 50  0001 C CNN
-F 1 "GND" H 9650 5750 50  0000 C CNN
-F 2 "" H 9650 5900 50  0001 C CNN
-F 3 "" H 9650 5900 50  0001 C CNN
-	1    9650 5900
-	1    0    0    -1
-$EndComp
-$Comp
 L Conn_01x06 J8
 U 1 1 5AA30710
@@
 	5400 1950 5600 1950
 Wire Wire Line
-	8700 1300 8100 1300
-Wire Wire Line
-	8700 1200 8550 1200
-Wire Wire Line
-	8550 1200 8550 1000
-Wire Wire Line
-	8700 1700 8550 1700
-Wire Wire Line
-	8700 1600 8550 1600
-Wire Wire Line
-	8700 1500 8550 1500
-Wire Wire Line
-	8700 1400 8550 1400
+	8350 1250 7750 1250
+Wire Wire Line
+	8350 1150 8200 1150
+Wire Wire Line
+	8200 1150 8200 950
+Wire Wire Line
+	8350 1650 8200 1650
+Wire Wire Line
+	8350 1550 8200 1550
+Wire Wire Line
+	8350 1450 8200 1450
+Wire Wire Line
+	8350 1350 8200 1350
 Wire Wire Line
 	9600 4450 9750 4450
@@
 Wire Notes Line
 	10650 6150 7350 6150
-Wire Wire Line
-	9650 3600 9650 3700
-Wire Wire Line
-	9650 4000 9650 4100
-Wire Wire Line
-	9650 4400 9650 4450
-Connection ~ 9650 4450
-Wire Wire Line
-	9650 5100 9650 5050
-Connection ~ 9650 5050
-Wire Wire Line
-	9650 5500 9650 5400
-Wire Wire Line
-	9650 5900 9650 5800
 Wire Wire Line
 	9900 1400 9850 1400
@@
 	1    0    0    -1
 $EndComp
-$Comp
-L VCC #PWR?
-U 1 1 5AAD9DC7
-P 9650 3600
-F 0 "#PWR?" H 9650 3450 50  0001 C CNN
-F 1 "VCC" H 9650 3750 50  0000 C CNN
-F 2 "" H 9650 3600 50  0001 C CNN
-F 3 "" H 9650 3600 50  0001 C CNN
-	1    9650 3600
-	1    0    0    -1
-$EndComp

Commit message: power board
Parts:
- removed J3: serial0, Pin_Headers:Pin_Header_Straight_1x04_Pitch2.54mm, symbol Conn_01x04
- removed J4: I2C, Pin_Headers:Pin_Header_Straight_1x04_Pitch2.54mm, symbol Conn_01x04
- removed J5: SPI 3V3, Pin_Headers:Pin_Header_Straight_1x06_Pitch2.54mm, symbol Conn_01x06
- removed J8: USB SER 3V3, Pin_Headers:Pin_Header_Straight_1x06_Pitch2.54mm, symbol Conn_01x06
- removed J9: DATA 5V, Pin_Headers:Pin_Header_Straight_1x02_Pitch2.54mm, symbol Conn_01x02
- added J3: Power 5V/5A, Pin_Headers:Pin_Header_Straight_1x05_Pitch2.54mm, symbol Conn_01x05
- added J6: Power/Data Input, Connectors_Molex:Molex_SPOX-5267_22-03-5035_03x2.54mm_Straight, symbol Conn_01x03
Connections:
- net +3V3: now also Q1.1 (G), R3.1
- net +5V: now also J3.1 (Pin_1)
- net DATA: now also J6.1 (Pin_1)
- net DTR: now also J1.11 (GPIO17_(GEN0))
- net GND: now also J3.2 (Pin_2), J3.3 (Pin_3), J6.3 (Pin_3)
- net IMU-RST: now also J1.13 (GPIO27_(GEN2)); no longer J1.29 (GPIO5)
- net RXI: now also J1.10 ((RXD0)_GPIO15), U2.4; no longer U3.4
- net TXO: now also J1.8 ((TXD0)_GPIO14), U3.2; no longer U2.2
- net VCC: no longer Q1.1 (G), R3.1
- net at Q1.2 (S), R3.2: now also U2.2, U3.4; no longer U2.4, U3.2
- net CS: no longer names the net of J1.24 ((~SPI_CE0~)_GPIO8)
- net MISO: no longer names the net of J1.21 ((SPI_MISO)_GPIO9)
- net MOSI: no longer names the net of J1.19 ((SPI_MOSI)_GPIO10)
- net SPI-CLK: no longer names the net of J1.23 ((SPI_SCLK)_GPIO11)
- new net +12V: J3.4 (Pin_4), J6.2 (Pin_2)
- no-connect marks 21 -> 23
Other:
- note removed: "GND\nCTS\n3V3\nTXO\nRXI\nDTR"
- moved on the sheet: J7, U2, U3
