File: ax12/electrical/rpi/robot.kicad_pcb (KiCad board)
At the start: 2 copper layers, 99.1 x 47 mm, 38 parts, among them J1 12V, J2 LEG1, J3 Pi USB Pwr, J4 Serial, J5 LEG2, J6 LEG3, J7 LEG4, J8 Data P, J9 Data S, U1 LM317_12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

Commit message: update
Parts:
- removed C3, C4: .1, Capacitors_THT:CP_Radial_D6.3mm_P2.50mm
- removed C5, C6: C, Capacitors_SMD:C_1206_HandSoldering
- removed J8: Data P, Pin_Headers:Pin_Header_Straight_1x03_Pitch2.54mm
- removed J9: Data S, Pin_Headers:Pin_Header_Straight_1x03_Pitch2.54mm
- removed R5: 10k, Resistors_SMD:R_1206_HandSoldering
- removed R6, R7, R8: 330, Resistors_SMD:R_1206_HandSoldering
- removed REF1, REF2, REF3, REF5, REF6, REF7, REF8: , Mounting_Holes:MountingHole_3.2mm_M3
- removed REF4: 3.2mm_M3, Mounting_Holes:MountingHole_3.2mm_M3
- removed U3: 74LS126, Housings_SOIC:SOIC-14_3.9x8.7mm_Pitch1.27mm
- removed U4: LM317_34, TO_SOT_Packages_THT:TO-220-3_Horizontal
- C1, C2: moved to F.Cu
- D1: value TX -> PWR; footprint LEDs:LED_D5.0mm -> LEDs:LED_1206_HandSoldering; moved to B.Cu
- D2: value RX -> TX; footprint LEDs:LED_D5.0mm -> LEDs:LED_1206_HandSoldering; moved to B.Cu
- D3: value PWR -> RX; moved to B.Cu
- J1: value 12V -> (none); footprint TerminalBlocks_Phoenix:TerminalBlock_Phoenix_PT-3.5mm_2pol -> Pin_Headers:Pin_Header_Straight_2x20_Pitch2.54mm; moved to B.Cu
- J2: value LEG1 -> IMU; footprint Connectors_Molex:Molex_MicroLatch-53253-0370_03x2.00mm_Straight -> Pin_Headers:Pin_Header_Straight_1x04_Pitch2.54mm
- J3: value Pi USB Pwr -> Lidar; footprint Pin_Headers:Pin_Header_Straight_1x02_Pitch2.54mm -> Pin_Headers:Pin_Header_Straight_1x04_Pitch2.54mm
- J5: value LEG2 -> Data S; footprint Connectors_Molex:Molex_MicroLatch-53253-0370_03x2.00mm_Straight -> Pin_Headers:Pin_Header_Straight_1x03_Pitch2.54mm
- J6: value LEG3 -> Pi USB Pwr; footprint Connectors_Molex:Molex_MicroLatch-53253-0370_03x2.00mm_Straight -> Pin_Headers:Pin_Header_Straight_1x02_Pitch2.54mm
- J7: value LEG4 -> Audio; footprint Connectors_Molex:Molex_MicroLatch-53253-0370_03x2.00mm_Straight -> Pin_Headers:Pin_Header_Straight_1x05_Pitch2.54mm
- R2: value 1.8k -> 10k; moved to F.Cu
- R4: value 1.8k -> 330
- U1: value LM317_12 -> AP1117-50; footprint TO_SOT_Packages_THT:TO-220-3_Horizontal -> TO_SOT_Packages_SMD:SOT-223-3_TabPin2
- U2: value AP1117-50 -> 74LS126; footprint TO_SOT_Packages_SMD:SOT-223-3_TabPin2 -> Housings_SOIC:SOIC-14_3.9x8.7mm_Pitch1.27mm; moved to F.Cu
- moved J4 91.9 mm to (153.0, 92.7)
- moved J1 46.2 mm to (111.8, 110.5), turned to 0 degrees
- moved D2 44.7 mm to (127.6, 78.7)
- moved J3 44.6 mm to (153.0, 109.9)
- moved J6 40.5 mm to (139.1, 62.2), turned to 270 degrees
- moved J7 40.4 mm to (152.4, 73.7), turned to 180 degrees
- moved D1 36.9 mm to (120.0, 71.8), turned to 270 degrees
- moved J5 34.5 mm to (146.1, 68.6), turned to 180 degrees
- moved U2 28.3 mm to (132.1, 92.1)
- moved D3 26.8 mm to (127.6, 82.5), turned to 0 degrees
- moved U1 25.9 mm to (128.3, 64.8), turned to 90 degrees
- moved J2 22.2 mm to (121.9, 110.5)
- moved R1 16.7 mm to (120.0, 81.3), turned to 90 degrees
- moved R2 15.8 mm to (123.2, 92.1)
- moved R3 14.8 mm to (135.9, 78.7), turned to 0 degrees
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Connections:
- C1 pad 2: GNDA -> GND
- C2 pad 2: GNDA -> GND
- D3 pad 1: GNDA -> GND
- J1 pad 1: GNDA -> Net-(J1-Pad1)
- J1 pad 2: +12V -> Net-(J1-Pad2)
- J2 pad 1: GNDA -> Net-(J1-Pad17)
- J2 pad 2: /PWR12 -> Net-(J1-Pad3)
- J2 pad 3: /DATA -> Net-(J1-Pad5)
- J3 pad 1: GNDA -> +5V
- J3 pad 2: +5V -> Net-(J1-Pad8)
- J5 pad 1: GNDA -> GND
- J5 pad 2: /PWR12 -> Net-(J5-Pad2)
- J5 pad 3: /DATA -> +12V
- J6 pad 1: GNDA -> GND
- J6 pad 2: /PWR34 -> +5V
- J7 pad 1: GNDA -> Net-(J7-Pad1)
- J7 pad 2: /PWR34 -> Net-(J7-Pad2)
- J7 pad 3: /DATA -> Net-(J7-Pad3)
- R1 pad 1: /PWR12 -> +5V
- R1 pad 2: Net-(R1-Pad2) -> Net-(D1-Pad2)
- R2 pad 1: Net-(R1-Pad2) -> +5V
- R2 pad 2: GNDA -> Net-(R2-Pad2)
- R3 pad 1: /PWR34 -> Net-(D2-Pad2)
- R3 pad 2: Net-(R3-Pad2) -> /TXI
- R4 pad 1: Net-(R3-Pad2) -> Net-(D3-Pad2)
- R4 pad 2: GNDA -> /RXO
- U1 pad 1: Net-(R1-Pad2) -> GND
- U1 pad 2: +12V -> +5V
- U1 pad 3: /PWR12 -> +12V
- U2 pad 1: GNDA -> /DTR
- U2 pad 2: +5V -> Net-(J5-Pad2)
- U2 pad 3: +12V -> /RXO
Routing:
- net GNDA: track 157.3 -> 0.00 mm, vias 1 -> 0
- net +12V: track 71.5 -> 0.00 mm, vias 2 -> 0
- net /RXO: track 51.3 -> 0.00 mm, vias 1 -> 0
- net +5V: track 49.5 -> 0.00 mm, vias 2 -> 0
- net GND: track 49.4 -> 0.00 mm, vias 3 -> 0
- net /DATA: track 48.8 -> 0.00 mm, vias 1 -> 0
- net /TXI: track 40.1 -> 0.00 mm
- net /PWR12: track 35.6 -> 0.00 mm
- net /PWR34: track 34.3 -> 0.00 mm
- net Net-(R5-Pad2): track 30.0 -> 0.00 mm
- net Net-(J9-Pad2): track 29.4 -> 0.00 mm, vias 1 -> 0
- net /DTR: track 22.8 -> 0.00 mm, vias 1 -> 0
- net Net-(R3-Pad2): track 19.7 -> 0.00 mm
- net +5VA: track 17.6 -> 0.00 mm, vias 1 -> 0
- net Net-(R1-Pad2): track 9.24 -> 0.00 mm
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Other:
- board size 99.1 x 47 mm -> 47 x 53.3 mm

Commit message: electrical update
Parts:
- added J8: SERIAL, Pin_Headers:Pin_Header_Straight_1x06_Pitch2.54mm, F.Cu at (113.0, 63.5)
- added J9: PWR BOARD, Pin_Headers:Pin_Header_Straight_1x03_Pitch2.54mm, F.Cu at (113.0, 82.5)
- added Q1: BSS138, TO_SOT_Packages_SMD:SOT-23, F.Cu at (139.7, 100.3)
- added R5: 330, Resistors_SMD:R_1206_HandSoldering, F.Cu at (120.7, 101.6)
- added REF**: MountingHole_2.7mm, Mounting_Holes:MountingHole_2.7mm, F.Cu at (113.0, 115.6)
- added REF**: MountingHole_2.7mm, Mounting_Holes:MountingHole_2.7mm, F.Cu at (113.0, 57.1)
- added REF**: MountingHole_2.7mm, Mounting_Holes:MountingHole_2.7mm, F.Cu at (160.0, 115.6)
- added REF**: MountingHole_2.7mm, Mounting_Holes:MountingHole_2.7mm, F.Cu at (160.0, 57.1)
- added U3: 74LVC1G126, TO_SOT_Packages_SMD:SOT-23-5_HandSoldering, F.Cu at (130.8, 100.3)
- D1, R1: moved to F.Cu
- J1: value (none) -> Raspberry_Pi_2_3; moved to F.Cu
- J2: footprint Pin_Headers:Pin_Header_Straight_1x04_Pitch2.54mm -> Pin_Headers:Pin_Header_Straight_1x06_Pitch2.54mm
- J4: value Serial -> I2C
- J5: value Data S -> SPI; footprint Pin_Headers:Pin_Header_Straight_1x03_Pitch2.54mm -> Pin_Headers:Pin_Header_Straight_1x06_Pitch2.54mm
- J7: footprint Pin_Headers:Pin_Header_Straight_1x05_Pitch2.54mm -> Pin_Headers:Pin_Header_Straight_1x07_Pitch2.54mm
- R2: value 10k -> 330
- U2: value 74LS126 -> 74LVC1G125; footprint Housings_SOIC:SOIC-14_3.9x8.7mm_Pitch1.27mm -> TO_SOT_Packages_SMD:SOT-23-5_HandSoldering
- moved J1 67.4 mm to (158.8, 62.2)
- moved J3 53.3 mm to (144.8, 57.1), turned to 270 degrees
- moved J7 53.1 mm to (113.0, 109.2)
- moved J4 23.3 mm to (148.6, 115.6), turned to 270 degrees
- moved U1 23.0 mm to (151.1, 67.3)
- moved J5 18.1 mm to (132.1, 57.1), turned to 270 degrees
- moved J2 5.68 mm to (119.4, 115.6)
- moved D1 4.49 mm to (120.7, 67.3), turned to 90 degrees
- moved J6 2.62 mm to (139.7, 64.8)
- moved R1 0.64 mm to (120.7, 81.3), turned to 270 degrees
Connections:
- D2 pad 1: GND -> Net-(D2-Pad1)
- D2 pad 2: Net-(D2-Pad2) -> +3V3
- D3 pad 1: GND -> Net-(D3-Pad1)
- D3 pad 2: Net-(D3-Pad2) -> RXI
- J1 pad 1: Net-(J1-Pad1) -> +3V3
- J1 pad 12: Net-(J1-Pad12) -> BCLK
- J1 pad 19: Net-(J1-Pad19) -> MOSI
- J1 pad 21: Net-(J1-Pad21) -> MISO
- J1 pad 23: Net-(J1-Pad23) -> SPI-CLK
- J1 pad 24: Net-(J1-Pad24) -> CS
- J1 pad 29: Net-(J1-Pad29) -> IMU-RST
- J1 pad 35: Net-(J1-Pad35) -> LRC
- J1 pad 40: Net-(J1-Pad40) -> DIN
- J2 pad 1: Net-(J1-Pad17) -> +3V3
- J2 pad 2: Net-(J1-Pad3) -> Net-(J2-Pad2)
- J2 pad 3: Net-(J1-Pad5) -> GND
- J2 pad 4: GND -> Net-(J1-Pad5)
- J4 pad 1: GND -> +3V3
- J4 pad 2: /DTR -> GND
- J4 pad 3: /RXO -> Net-(J1-Pad3)
- J4 pad 4: /TXI -> Net-(J1-Pad5)
- J5 pad 1: GND -> +3V3
- J5 pad 2: Net-(J5-Pad2) -> GND
- J5 pad 3: +12V -> CS
- J7 pad 1: Net-(J7-Pad1) -> LRC
- J7 pad 2: Net-(J7-Pad2) -> BCLK
- J7 pad 3: Net-(J7-Pad3) -> DIN
- R2 pad 2: Net-(R2-Pad2) -> DATA
- R3 pad 1: Net-(D2-Pad2) -> +3V3
- R3 pad 2: /TXI -> DTR
- R4 pad 1: Net-(D3-Pad2) -> Net-(D2-Pad1)
- R4 pad 2: /RXO -> TXO
- U2 pad 1: /DTR -> DTR
- U2 pad 2: Net-(J5-Pad2) -> TXO
- U2 pad 3: /RXO -> GND
- U2 pad 4: /DTR -> DTR
- U2 pad 5: GND -> +3V3
Other:
- board size 47 x 53.3 mm -> 54.6 x 63.5 mm

Commit message: update
Parts:
- removed C1, C2: C, Capacitors_SMD:C_1206_HandSoldering
- removed D1: PWR, LEDs:LED_1206_HandSoldering
- removed J6: Pi USB Pwr, Pin_Headers:Pin_Header_Straight_1x02_Pitch2.54mm
- removed R1: 330, Resistors_SMD:R_1206_HandSoldering
- removed U1: AP1117-50, TO_SOT_Packages_SMD:SOT-223-3_TabPin2
- D2, D3, R4: moved to F.Cu
- J3: value Lidar -> serial0
- J8: value SERIAL -> USB SER 3V3
- J9: value PWR BOARD -> DATA 5V; footprint Pin_Headers:Pin_Header_Straight_1x03_Pitch2.54mm -> Pin_Headers:Pin_Header_Straight_1x02_Pitch2.54mm
- Q1, U2, U3: moved to B.Cu
- R2: value 330 -> 10k; moved to B.Cu
- R3: value 330 -> 10k
- moved J4 63.8 mm to (111.8, 63.5), turned to 0 degrees
- moved J2 57.2 mm to (120.7, 58.4)
- moved D2 38.9 mm to (146.1, 113.0), turned to 90 degrees
- moved J9 34.9 mm to (147.3, 88.9), turned to 270 degrees
- moved J8 33.0 mm to (111.8, 96.5)
- moved R2 32.8 mm to (151.1, 109.2), turned to 180 degrees
- moved D3 31.6 mm to (135.9, 113.0), turned to 90 degrees
- moved R4 30.9 mm to (141.0, 113.0), turned to 90 degrees
- moved J5 27.9 mm to (150.5, 78.1), turned to 180 degrees
- moved J7 17.8 mm to (111.8, 91.4)
- moved R3 17.8 mm to (134.6, 96.5)
- moved U2 16.7 mm to (144.8, 102.9), turned to 0 degrees
- moved R5 15.3 mm to (130.8, 113.0), turned to 90 degrees
- moved Q1 11.7 mm to (151.1, 102.9)
- moved J3 6.48 mm to (151.1, 58.4)
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Connections:
- J1 pad 4: Net-(J1-Pad4) -> +5V
- J9 pad 2: +12V -> GND
- Q1 pad 2: DTR -> Net-(Q1-Pad2)
- R3 pad 2: DTR -> Net-(Q1-Pad2)
- U2 pad 4: DTR -> Net-(Q1-Pad2)
- U3 pad 2: DTR -> Net-(Q1-Pad2)
Other:
- board size 54.6 x 63.5 mm -> 55.9 x 63.5 mm
- board text added: "GND DATA"

Commit message: power board
Parts:
- removed D2: TX, LEDs:LED_1206_HandSoldering
- removed D3: RX, LEDs:LED_1206_HandSoldering
- removed J4: I2C, Pin_Headers:Pin_Header_Straight_1x04_Pitch2.54mm
- removed J5: SPI, Pin_Headers:Pin_Header_Straight_1x06_Pitch2.54mm
- removed J8: USB SER 3V3, Pin_Headers:Pin_Header_Straight_1x06_Pitch2.54mm
- removed J9: DATA 5V, Pin_Headers:Pin_Header_Straight_1x02_Pitch2.54mm
- removed R4, R5: 330, Resistors_SMD:R_1206_HandSoldering
- removed REF** (x4): MountingHole_2.7mm, Mounting_Holes:MountingHole_2.7mm
- added J6: Power/Data Input, Connectors_Molex:Molex_SPOX-5267_22-03-5035_03x2.54mm_Straight, F.Cu at (135.9, 109.9)
- added REF***: , Symbols:OSHW-Logo_7.5x8mm_SilkScreen, F.Cu at (149.2, 103.5)
- J3: value serial0 -> Power 5V/5A; footprint Pin_Headers:Pin_Header_Straight_1x04_Pitch2.54mm -> Pin_Headers:Pin_Header_Straight_1x05_Pitch2.54mm
- moved J3 37.9 mm to (136.5, 93.3), turned to 0 degrees
- moved U2 37.2 mm to (149.9, 66.0), turned to 180 degrees
- moved U3 32.4 mm to (149.9, 73.7), turned to 180 degrees
- moved J7 24.9 mm to (136.5, 88.9)
- moved R3 22.0 mm to (149.9, 80.6)
- moved J2 19.2 mm to (136.5, 69.2), turned to 180 degrees
- moved Q1 15.3 mm to (149.9, 87.6), turned to 270 degrees
- moved R2 15.3 mm to (150.5, 94.0), turned to 0 degrees
Connections:
- J1 pad 10: Net-(J1-Pad10) -> RXI
- J1 pad 11: Net-(J1-Pad11) -> DTR
- J1 pad 13: Net-(J1-Pad13) -> IMU-RST
- J1 pad 15: Net-(J1-Pad15) -> (no net)
- J1 pad 16: Net-(J1-Pad16) -> (no net)
- J1 pad 17: Net-(J1-Pad17) -> VCC
- J1 pad 18: Net-(J1-Pad18) -> (no net)
- J1 pad 19: MOSI -> (no net)
- J1 pad 2: Net-(J1-Pad2) -> +5V
- J1 pad 21: MISO -> (no net)
- J1 pad 22: Net-(J1-Pad22) -> (no net)
- J1 pad 23: SPI-CLK -> (no net)
- J1 pad 24: CS -> (no net)
- J1 pad 26: Net-(J1-Pad26) -> (no net)
- J1 pad 27: Net-(J1-Pad27) -> (no net)
- J1 pad 28: Net-(J1-Pad28) -> (no net)
- J1 pad 29: IMU-RST -> (no net)
- J1 pad 31: Net-(J1-Pad31) -> (no net)
- J1 pad 32: Net-(J1-Pad32) -> (no net)
- J1 pad 33: Net-(J1-Pad33) -> (no net)
- J1 pad 36: Net-(J1-Pad36) -> (no net)
- J1 pad 37: Net-(J1-Pad37) -> (no net)
- J1 pad 38: Net-(J1-Pad38) -> (no net)
- J1 pad 7: Net-(J1-Pad7) -> (no net)
- J1 pad 8: Net-(J1-Pad8) -> TXO
- J2 pad 2: Net-(J2-Pad2) -> (no net)
- J3 pad 2: Net-(J1-Pad8) -> GND
- J3 pad 3: Net-(J1-Pad10) -> GND
- J3 pad 4: GND -> +12V
- J7 pad 4: Net-(J7-Pad4) -> (no net)
- J7 pad 5: Net-(J7-Pad5) -> (no net)
- U2 pad 2: TXO -> Net-(Q1-Pad2)
- U2 pad 4: Net-(Q1-Pad2) -> RXI
- U2 pad 5: +3V3 -> VCC
- U3 pad 2: Net-(Q1-Pad2) -> TXO
- U3 pad 4: RXI -> Net-(Q1-Pad2)
- U3 pad 5: +3V3 -> VCC
Routing:
- net +5V: track 0.00 -> 78.1 mm, vias 0 -> 1
- net +3V3: track 0.00 -> 51.5 mm, vias 0 -> 5
- net GND: track 0.00 -> 51.0 mm, vias 0 -> 1
- net IMU-RST: track 0.00 -> 46.5 mm, vias 0 -> 1
- net DIN: track 0.00 -> 41.3 mm, vias 0 -> 2
- net BCLK: track 0.00 -> 40.2 mm, vias 0 -> 2
- net Net-(Q1-Pad2): track 0.00 -> 32.4 mm, vias 0 -> 2
- net DATA: track 0.00 -> 31.4 mm
- net LRC: track 0.00 -> 29.1 mm, vias 0 -> 1
- net VCC: track 0.00 -> 28.5 mm, vias 0 -> 1
- net Net-(J1-Pad3): track 0.00 -> 24.6 mm
- net Net-(J1-Pad5): track 0.00 -> 24.6 mm
- net DTR: track 0.00 -> 20.5 mm
- net +12V: track 0.00 -> 20.4 mm
- net RXI: track 0.00 -> 20.0 mm, vias 0 -> 1
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- added copper zone on B.Cu, net GND
- added copper zone on F.Cu, net GND
Other:
- board size 55.9 x 63.5 mm -> 29.8 x 63.5 mm
- board text added: "Kevin Walchko Ver. 1 (c) 2018"
- board text removed: "GND DATA"

Commit message: updated pi board
Parts:
- added J4: i2c, Pin_Headers:Pin_Header_Straight_1x04_Pitch2.54mm, F.Cu at (151.8, 56.5)
Routing:
- net IMU-RST: track 46.5 -> 36.9 mm, vias 1 -> 6
- net Net-(J1-Pad5): track 24.6 -> 30.0 mm
- net +3V3: track 51.5 -> 55.6 mm
- net Net-(J1-Pad3): track 24.6 -> 26.7 mm
Changed lines of the file:
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@@
 (kicad_pcb (version 4) (host pcbnew 4.0.7)
   (general
-    (links 39)
+    (links 43)
     (no_connects 0)
     (area 123.64119 54.489999 163.905001 119.285477)
     (thickness 1.6)
     (drawings 7)
-    (tracks 167)
+    (tracks 182)
     (zones 0)
-    (modules 11)
+    (modules 12)
     (nets 17)
   )
@@
       (xy 0.500964 -3.601424)) (layer F.SilkS) (width 0.01))
   )
+  (module Pin_Headers:Pin_Header_Straight_1x04_Pitch2.54mm (layer F.Cu)
+    (at 151.765 56.515 270)
+    (descr "Through hole straight pin header, 1x04, 2.54mm pitch, single row")
+    (tags "Through hole pin header THT 1x04 2.54mm single row")
+    (fp_text reference J4 (at 0 -2.33 270) (layer F.SilkS)
+      (effects (font (size 1 1) (thickness 0.15)))
+    )
+    (fp_text value i2c (at 0 9.95 270) (layer F.Fab)
+      (effects (font (size 1 1) (thickness 0.15)))
+    )
+    (fp_line (start -0.635 -1.27) (end 1.27 -1.27) (layer F.Fab) (width 0.1))
+    (fp_line (start 1.27 -1.27) (end 1.27 8.89) (layer F.Fab) (width 0.1))
+    (fp_line (start 1.27 8.89) (end -1.27 8.89) (layer F.Fab) (width 0.1))
+    (fp_line (start -1.27 8.89) (end -1.27 -0.635) (layer F.Fab) (width 0.1))
+    (fp_line (start -1.27 -0.635) (end -0.635 -1.27) (layer F.Fab) (width 0.1))
+    (fp_line (start -1.33 8.95) (end 1.33 8.95) (layer F.SilkS) (width 0.12))
+    (fp_line (start -1.33 1.27) (end -1.33 8.95) (layer F.SilkS) (width 0.12))
+    (fp_line (start 1.33 1.27) (end 1.33 8.95) (layer F.SilkS) (width 0.12))
+    (fp_line (start -1.33 1.27) (end 1.33 1.27) (layer F.SilkS) (width 0.12))
+    (fp_line (start -1.33 0) (end -1.33 -1.33) (layer F.SilkS) (width 0.12))
+    (fp_line (start -1.33 -1.33) (end 0 -1.33) (layer F.SilkS) (width 0.12))
+    (fp_line (start -1.8 -1.8) (end -1.8 9.4) (layer F.CrtYd) (width 0.05))
+    (fp_line (start -1.8 9.4) (end 1.8 9.4) (layer F.CrtYd) (width 0.05))
+    (fp_line (start 1.8 9.4) (end 1.8 -1.8) (layer F.CrtYd) (width 0.05))
+    (fp_line (start 1.8 -1.8) (end -1.8 -1.8) (layer F.CrtYd) (width 0.05))
+    (fp_text user %R (at 0 3.81 360) (layer F.Fab)
+      (effects (font (size 1 1) (thickness 0.15)))
+    )
+    (pad 1 thru_hole rect (at 0 0 270) (size 1.7 1.7) (drill 1) (layers *.Cu *.Mask)
+      (net 5 +3V3))
+    (pad 2 thru_hole oval (at 0 2.54 270) (size 1.7 1.7) (drill 1) (layers *.Cu *.Mask)
+      (net 1 GND))
+    (pad 3 thru_hole oval (at 0 5.08 270) (size 1.7 1.7) (drill 1) (layers *.Cu *.Mask)
+      (net 3 "Net-(J1-Pad3)"))
+    (pad 4 thru_hole oval (at 0 7.62 270) (size 1.7 1.7) (drill 1) (layers *.Cu *.Mask)
+      (net 4 "Net-(J1-Pad5)"))
+    (model ${KISYS3DMOD}/Pin_Headers.3dshapes/Pin_Header_Straight_1x04_Pitch2.54mm.wrl
+      (at (xyz 0 0 0))
+      (scale (xyz 1 1 1))
+      (rotate (xyz 0 0 0))
+    )
+  )
   (gr_text "Kevin Walchko\nVer. 1\n(c) 2018" (at 147.955 113.665) (layer F.SilkS)
     (effects (font (size 1.5 1.5) (thickness 0.3)))
@@
   (segment (start 149.86 71.755) (end 149.86 65.405) (width 1.6) (layer F.Cu) (net 2))
   (segment (start 144.78 93.345) (end 149.86 88.265) (width 1.6) (layer F.Cu) (net 2))
-  (segment (start 158.75 64.77) (end 155.575 64.77) (width 0.25) (layer B.Cu) (net 3))
-  (segment (start 149.86 59.055) (end 136.525 59.055) (width 0.25) (layer B.Cu) (net 3))
-  (segment (start 155.575 64.77) (end 149.86 59.055) (width 0.25) (layer B.Cu) (net 3))
+  (segment (start 136.525 59.055) (end 144.145 59.055) (width 0.25) (layer F.Cu) (net 3))
+  (segment (start 144.145 59.055) (end 146.685 56.515) (width 0.25) (layer F.Cu) (net 3))
+  (segment (start 146.685 56.515) (end 151.13 60.96) (width 0.25) (layer B.Cu) (net 3))
+  (segment (start 156.845 64.77) (end 158.75 64.77) (width 0.25) (layer B.Cu) (net 3))
+  (segment (start 153.035 60.96) (end 156.845 64.77) (width 0.25) (layer B.Cu) (net 3))
+  (segment (start 151.13 60.96) (end 153.035 60.96) (width 0.25) (layer B.Cu) (net 3))
+  (segment (start 144.145 56.515) (end 144.145 59.69) (width 0.25) (layer B.Cu) (net 4))
+  (segment (start 144.145 59.69) (end 145.415 62.23) (width 0.25) (layer B.Cu) (net 4))
   (segment (start 158.75 67.31) (end 156.845 67.31) (width 0.25) (layer B.Cu) (net 4))
-  (segment (start 151.13 61.595) (end 136.525 61.595) (width 0.25) (layer B.Cu) (net 4))
-  (segment (start 156.845 67.31) (end 151.13 61.595) (width 0.25) (layer B.Cu) (net 4))
+  (segment (start 150.495 62.23) (end 145.415 62.23) (width 0.25) (layer B.Cu) (net 4))
+  (segment (start 145.415 62.23) (end 136.525 61.595) (width 0.25) (layer B.Cu) (net 4))
+  (segment (start 156.845 67.31) (end 150.495 62.23) (width 0.25) (layer B.Cu) (net 4))
+  (segment (start 151.765 56.515) (end 151.765 59.69) (width 0.25) (layer B.Cu) (net 5))
+  (segment (start 151.765 59.69) (end 152.4 60.325) (width 0.25) (layer B.Cu) (net 5))
   (segment (start 147.86 80.645) (end 144.145 80.645) (width 0.25) (layer B.Cu) (net 5))
   (via (at 144.145 80.645) (size 0.6) (drill 0.4) (layers F.Cu B.Cu) (net 5))
@@
   (segment (start 156.845 76.2) (end 155.575 77.47) (width 0.25) (layer B.Cu) (net 7))
   (segment (start 160.02 76.2) (end 156.845 76.2) (width 0.25) (layer B.Cu) (net 7))
-  (segment (start 158.75 77.47) (end 156.21 74.93) (width 0.25) (layer F.Cu) (net 8) (status 80000))
-  (segment (start 156.21 74.93) (end 156.21 70.485) (width 0.25) (layer F.Cu) (net 8) (status 80000))
-  (segment (start 156.21 70.485) (end 155.575 69.85) (width 0.25) (layer F.Cu) (net 8) (status 80000))
-  (segment (start 155.575 69.85) (end 155.575 69.215) (width 0.25) (layer F.Cu) (net 8) (status 80000))
-  (via (at 155.575 69.215) (size 0.6) (layers F.Cu B.Cu) (net 8) (status 80000))
-  (segment (start 155.575 69.215) (end 156.21 68.58) (width 0.25) (layer B.Cu) (net 8) (status 80000))
-  (segment (start 156.21 68.58) (end 160.02 68.58) (width 0.25) (layer B.Cu) (net 8) (status 80000))
-  (segment (start 160.02 68.58) (end 160.02 63.5) (width 0.25) (layer B.Cu) (net 8) (status 80000))
-  (segment (start 160.02 63.5) (end 157.48 63.5) (width 0.25) (layer B.Cu) (net 8) (status 80000))
-  (segment (start 157.48 63.5) (end 157.48 62.23) (width 0.25) (layer B.Cu) (net 8) (status 80000))
-  (segment (start 157.48 62.23) (end 151.765 56.515) (width 0.25) (layer B.Cu) (net 8) (status 80000))
-  (segment (start 151.765 56.515) (end 136.525 56.515) (width 0.25) (layer B.Cu) (net 8) (status 80000))
+  (segment (start 136.525 56.515) (end 139.065 56.515) (width 0.25) (layer F.Cu) (net 8))
+  (segment (start 156.845 75.565) (end 158.75 77.47) (width 0.25) (layer F.Cu) (net 8))
+  (segment (start 156.845 71.12) (end 156.845 75.565) (width 0.25) (layer F.Cu) (net 8))
+  (segment (start 155.575 69.85) (end 156.845 71.12) (width 0.25) (layer F.Cu) (net 8))
+  (via (at 155.575 69.85) (size 0.6) (drill 0.4) (layers F.Cu B.Cu) (net 8))
+  (segment (start 155.575 67.31) (end 155.575 69.85) (width 0.25) (layer B.Cu) (net 8))
+  (via (at 155.575 67.31) (size 0.6) (drill 0.4) (layers F.Cu B.Cu) (net 8))
+  (segment (start 155.575 64.77) (end 155.575 67.31) (width 0.25) (layer F.Cu) (net 8))
+  (via (at 155.575 64.77) (size 0.6) (drill 0.4) (layers F.Cu B.Cu) (net 8))
+  (segment (start 152.4 61.595) (end 155.575 64.77) (width 0.25) (layer B.Cu) (net 8))
+  (segment (start 147.32 61.595) (end 152.4 61.595) (width 0.25) (layer B.Cu) (net 8))
+  (segment (start 146.05 60.325) (end 147.32 61.595) (width 0.25) (layer B.Cu) (net 8))
+  (via (at 146.05 60.325) (size 0.6) (drill 0.4) (layers F.Cu B.Cu) (net 8))
+  (segment (start 142.24 60.325) (end 146.05 60.325) (width 0.25) (layer F.Cu) (net 8))
+  (via (at 142.24 60.325) (size 0.6) (drill 0.4) (layers F.Cu B.Cu) (net 8))
+  (segment (start 142.24 59.69) (end 142.24 60.325) (width 0.25) (layer B.Cu) (net 8))
+  (segment (start 140.335 57.785) (end 142.24 59.69) (width 0.25) (layer B.Cu) (net 8))
+  (via (at 140.335 57.785) (size 0.6) (drill 0.4) (layers F.Cu B.Cu) (net 8))
+  (segment (start 139.065 56.515) (end 140.335 57.785) (width 0.25) (layer F.Cu) (net 8))
   (segment (start 136.525 88.9) (end 144.145 96.52) (width 0.25) (layer B.Cu) (net 9) (status 80000))
   (segment (start 144.145 96.52) (end 149.86 96.52) (width 0.25) (layer B.Cu) (net 9) (status 80000))
